File: KiCad/Retificador_de_tenção.sch (KiCad schematic (older format))
At the start: 3 parts

Commit message: .
Parts:
- added D1: 1N5819, Diode_THT:D_DO-41_SOD81_P10.16mm_Horizontal, symbol Diode:1N5819
Connections:
- net in: now also D1.2 (A); no longer C1.1, Retificador_de_tensão_5v.2 (VIN)
- new net: C1.1, D1.1 (K), Retificador_de_tensão_5v.2 (VIN)
Changed lines of the file:
@@
 	1    0    0    -1
 $EndComp
-Text HLabel 3700 3300 0    50   Input ~ 0
+Text HLabel 3500 3300 0    50   Input ~ 0
 in
 Text HLabel 6250 3300 2    50   Output ~ 0
@@
 Connection ~ 6100 3300
 Wire Wire Line
-	3700 3300 4100 3300
-Wire Wire Line
 	4100 3300 4100 3500
-Connection ~ 4100 3300
 Wire Wire Line
 	4100 3300 4300 3300
@@
 Wire Wire Line
 	4300 3050 4100 3050
+$Comp
+L Diode:1N5819 D1
+U 1 1 60A5E713
+P 3750 3300
+F 0 "D1" H 3750 3083 50  0000 C CNN
+F 1 "1N5819" H 3750 3174 50  0000 C CNN
+F 2 "Diode_THT:D_DO-41_SOD81_P10.16mm_Horizontal" H 3750 3125 50  0001 C CNN
+F 3 "http://www.vishay.com/docs/88525/1n5817.pdf" H 3750 3300 50  0001 C CNN
+	1    3750 3300
+	-1   0    0    1
+$EndComp
+Wire Wire Line
+	3900 3300 4100 3300
+Connection ~ 4100 3300
+Wire Wire Line
+	3500 3300 3600 3300
 $EndSCHEMATC

Commit message: .
Parts:
- removed Retificador_de_tensão_5v: LD1117DT50TR, DPAK_STM, symbol 2021-05-14_18-10-03:LD1117DT50TR
- added Retificador_de_tensão_5v: LD1117DT50TR, DPAK_STM, symbol My_Lib:LD1117DT50TR
Connections:
- net GNDREF: now also Retificador_de_tensão_5v.1 (ADJ/GND)
- net out: now also Retificador_de_tensão_5v.3 (VOUT)
- net at C1.1, D1.1 (K): now also Retificador_de_tensão_5v.2 (VIN)
Changed lines of the file:
@@
 Wire Wire Line
 	5250 3800 5250 4050
-$Comp
-L 2021-05-14_18-10-03:LD1117DT50TR Retificador_de_tensão_5v
-U 1 1 60A15D94
-P 4300 3200
-F 0 "Retificador_de_tensão_5v" H 5200 3587 60  0000 C CNN
-F 1 "LD1117DT50TR" H 5200 3481 60  0000 C CNN
-F 2 "DPAK_STM" H 5200 3440 60  0001 C CNN
-F 3 "" H 4300 3200 60  0000 C CNN
-	1    4300 3200
-	1    0    0    -1
-$EndComp
 Wire Wire Line
 	5250 3800 6100 3800
@@
 	4100 3800 5250 3800
 Connection ~ 5250 3800
-Connection ~ 6100 3300
 Wire Wire Line
 	4100 3300 4100 3500
@@
 Wire Wire Line
 	3500 3300 3600 3300
+$Comp
+L My_Lib:LD1117DT50TR Retificador_de_tensão_5v
+U 1 1 60A5A48D
+P 4300 3200
+F 0 "Retificador_de_tensão_5v" H 5200 3587 60  0000 C CNN
+F 1 "LD1117DT50TR" H 5200 3481 60  0000 C CNN
+F 2 "DPAK_STM" H 5200 3440 60  0001 C CNN
+F 3 "" H 4300 3200 60  0000 C CNN
+	1    4300 3200
+	1    0    0    -1
+$EndComp
+Connection ~ 6100 3300
 $EndSCHEMATC
