File: KiCad/_autosave-Projeto_PBLE01.sch (KiCad schematic (older format))
At the start: 13 parts

Commit message: .
Parts:
- D_PWR_GREEN: renamed from D_PWR; value LED -> G_LED
- R_LED_PWR: value 15 -> 200
Connections:
- net labels added: CTS_Conversor
- wire segments 58 -> 60
Changed lines of the file:
@@
 $Descr A4 11693 8268
 encoding utf-8
-Sheet 1 3
+Sheet 1 4
 Title ""
 Date ""
@@
 VUSB_3.3v
 Text GLabel 7900 950  0    50   Input ~ 0
-VUSB_3.3v
+Vcc_5v
 Wire Wire Line
 	7900 950  8050 950
@@
 $EndComp
 $Comp
-L Device:LED D_PWR
+L Device:LED D_PWR_GREEN
 U 1 1 60A99312
 P 9050 5950
-F 0 "D_PWR" H 9043 5787 50  0000 C CNN
-F 1 "LED" H 9043 5786 50  0001 C CNN
+F 0 "D_PWR_GREEN" H 9043 5787 50  0000 C CNN
+F 1 "G_LED" H 9043 5786 50  0001 C CNN
 F 2 "" H 9050 5950 50  0001 C CNN
 F 3 "~" H 9050 5950 50  0001 C CNN
@@
 P 8700 5950
 F 0 "R_LED_PWR" V 8495 5950 50  0001 C CNN
-F 1 "15" V 8587 5950 50  0000 C CNN
+F 1 "200" V 8587 5950 50  0000 C CNN
 F 2 "" V 8740 5940 50  0001 C CNN
 F 3 "~" H 8700 5950 50  0001 C CNN
@@
 Wire Notes Line
 	700  6700 700  7600
+Text Label 7100 1700 2    50   ~ 0
+CTS_Conversor
+Text Label 4150 2450 0    50   ~ 0
+CTS_Conversor
+Wire Wire Line
+	4100 2450 4150 2450
+$Comp
+L power:GNDREF #PWR?
+U 1 1 60AAEC4B
+P 8500 950
+F 0 "#PWR?" H 8500 700 50  0001 C CNN
+F 1 "GNDREF" H 8505 777 50  0000 C CNN
+F 2 "" H 8500 950 50  0001 C CNN
+F 3 "" H 8500 950 50  0001 C CNN
+	1    8500 950
+	1    0    0    -1
+$EndComp
+$Sheet
+S 9200 2250 500  300
+U 60AB2F80
+F0 "Ocilador_Conversor" 50
+F1 "Ocilador_Conversor.sch" 50
+$EndSheet
+Wire Wire Line
+	7100 1700 7250 1700
 $EndSCHEMATC
