File: KiCad/Projeto_PBLE01.sch (KiCad schematic (older format))
At the start: 5 parts

Commit message: .
Parts:
- removed ICSP_Pins: Conn_01x03_Male, symbol Connector:Conn_01x03_Male
- removed U?: LM358, symbol Amplifier_Operational:LM358
- added ICSP_Pin: Conn_01x05_Male, symbol Connector:Conn_01x05_Male
Connections:
- net labels added: ICSP_MCLR, Serial_Clk, Serial_Data
- net labels removed: ICSP_Program_enable
- wire segments 21 -> 27
Other:
- note added: "Alimentação"
- note added: "PIC18F4550-I/PT"
- note added: "Saídas/entradas"
- moved on the sheet: J?
Changed lines of the file:
@@
 L Connector:USB_B J?
 U 1 1 609F2570
-P 1250 5450
-F 0 "J?" H 1307 5917 50  0000 C CNN
-F 1 "USB_B" H 1307 5826 50  0000 C CNN
-F 2 "" H 1400 5400 50  0001 C CNN
-F 3 " ~" H 1400 5400 50  0001 C CNN
-	1    1250 5450
-	1    0    0    -1
-$EndComp
-$Comp
-L Amplifier_Operational:LM358 U?
-U 1 1 609FD288
-P 4850 6450
-F 0 "U?" H 4850 6817 50  0000 C CNN
-F 1 "LM358" H 4850 6726 50  0000 C CNN
-F 2 "" H 4850 6450 50  0001 C CNN
-F 3 "http://www.ti.com/lit/ds/symlink/lm2904-n.pdf" H 4850 6450 50  0001 C CNN
-	1    4850 6450
+P 1200 5450
+F 0 "J?" H 1257 5917 50  0000 C CNN
+F 1 "USB_B" H 1257 5826 50  0000 C CNN
+F 2 "" H 1350 5400 50  0001 C CNN
+F 3 " ~" H 1350 5400 50  0001 C CNN
+	1    1200 5450
 	1    0    0    -1
 $EndComp
@@
 L power:GNDREF #PWR?
 U 1 1 60A478EE
-P 1250 6100
-F 0 "#PWR?" H 1250 5850 50  0001 C CNN
-F 1 "GNDREF" H 1255 5927 50  0000 C CNN
-F 2 "" H 1250 6100 50  0001 C CNN
-F 3 "" H 1250 6100 50  0001 C CNN
-	1    1250 6100
+P 1200 6100
+F 0 "#PWR?" H 1200 5850 50  0001 C CNN
+F 1 "GNDREF" H 1205 5927 50  0000 C CNN
+F 2 "" H 1200 6100 50  0001 C CNN
+F 3 "" H 1200 6100 50  0001 C CNN
+	1    1200 6100
 	1    0    0    -1
 $EndComp
@@
 	8150 2700 8150 2950
 Wire Wire Line
-	1250 6100 1250 5850
-Text GLabel 1850 5250 2    50   Input ~ 0
-Vcc_5v
-Wire Wire Line
-	1850 5250 1550 5250
+	1200 6100 1200 5850
+Text GLabel 1800 5250 2    50   Input ~ 0
+Vcc_5v
+Wire Wire Line
+	1800 5250 1500 5250
 Text GLabel 7950 950  0    50   Input ~ 0
 Vcc_5v
@@
 	8050 950  8050 1100
 $Sheet
-S 5000 1750 800  700
+S 5500 1500 800  400
 U 60A4FE38
 F0 "Timer_I2C" 50
 F1 "Timer_I2C.sch" 50
-F2 "X1_ocilador" B L 5000 2200 50
-F3 "X2_ocilador" B L 5000 2300 50
-F4 "Serial_CLK" I L 5000 2050 50
-F5 "Serial_DATA" B L 5000 1950 50
-F6 "Multifunction_pin" B L 5000 1800 50
+F2 "Serial_CLK" I L 5500 1800 50
+F3 "Serial_DATA" B L 5500 1700 50
+F4 "Multifunction_pin" B L 5500 1550 50
 $EndSheet
-$Comp
-L Connector:Conn_01x03_Male ICSP_Pins
-U 1 1 60A6D604
-P 2500 5400
-F 0 "ICSP_Pins" H 2608 5681 50  0000 C CNN
-F 1 "Conn_01x03_Male" H 2608 5590 50  0000 C CNN
-F 2 "" H 2500 5400 50  0001 C CNN
-F 3 "~" H 2500 5400 50  0001 C CNN
-	1    2500 5400
-	1    0    0    -1
-$EndComp
-Text Label 2950 5300 0    50   ~ 0
-ICSP_Program_enable
-Text Label 2950 5400 0    50   ~ 0
+Text Label 2900 5800 0    50   ~ 0
 ICSP_Clk
-Text Label 2950 5500 0    50   ~ 0
+Text Label 2900 5700 0    50   ~ 0
 ICSP_Data
-Wire Wire Line
-	2700 5300 2950 5300
-Wire Wire Line
-	2700 5400 2950 5400
-Wire Wire Line
-	2700 5500 2950 5500
-Text Label 1350 2950 2    50   ~ 0
-ICSP_Program_enable
 Text Label 1350 3050 2    50   ~ 0
 ICSP_Clk
@@
 ICSP_Data
 Wire Wire Line
-	1350 2950 1700 2950
-Wire Wire Line
 	1350 3050 1700 3050
 Wire Wire Line
 	1350 3150 1700 3150
+Text Label 4300 3650 0    50   ~ 0
+ICSP_MCLR
+Wire Wire Line
+	4100 3650 4300 3650
+$Comp
+L Connector:Conn_01x05_Male ICSP_Pin
+U 1 1 60A58DC0
+P 2450 5600
+F 0 "ICSP_Pin" H 2558 5981 50  0000 C CNN
+F 1 "Conn_01x05_Male" H 2558 5890 50  0000 C CNN
+F 2 "" H 2450 5600 50  0001 C CNN
+F 3 "~" H 2450 5600 50  0001 C CNN
+	1    2450 5600
+	1    0    0    -1
+$EndComp
+Wire Wire Line
+	2650 5400 2900 5400
+Text Label 2900 5400 0    50   ~ 0
+ICSP_MCLR
+Wire Wire Line
+	2900 5800 2650 5800
+Wire Wire Line
+	2650 5700 2900 5700
+$Comp
+L power:GNDREF #PWR?
+U 1 1 60A5C611
+P 3500 5600
+F 0 "#PWR?" H 3500 5350 50  0001 C CNN
+F 1 "GNDREF" H 3505 5427 50  0000 C CNN
+F 2 "" H 3500 5600 50  0001 C CNN
+F 3 "" H 3500 5600 50  0001 C CNN
+	1    3500 5600
+	1    0    0    -1
+$EndComp
+Text GLabel 3500 5500 2    50   Input ~ 0
+Vcc_5v
+Wire Wire Line
+	2650 5500 3500 5500
+Wire Wire Line
+	3500 5600 2650 5600
+Text Label 5350 1700 2    50   ~ 0
+Serial_Data
+Text Label 5350 1800 2    50   ~ 0
+Serial_Clk
+Wire Wire Line
+	5500 1800 5350 1800
+Wire Wire Line
+	5500 1700 5350 1700
+Text Label 1550 2450 2    50   ~ 0
+Serial_Data
+Text Label 1550 2550 2    50   ~ 0
+Serial_Clk
+Wire Wire Line
+	1700 2550 1550 2550
+Wire Wire Line
+	1700 2450 1550 2450
+Wire Notes Line
+	5950 4850 5950 6500
+Wire Notes Line
+	5950 6500 700  6500
+Wire Notes Line
+	700  6500 700  4850
+Wire Notes Line
+	700  4850 5950 4850
+Text Notes 750  4850 0    50   ~ 0
+Saídas/entradas
+Wire Notes Line
+	2750 6700 2750 7500
+Wire Notes Line
+	2750 7500 700  7500
+Wire Notes Line
+	700  7500 700  6700
+Wire Notes Line
+	700  6700 2750 6700
+Text Notes 750  6700 0    50   ~ 0
+Alimentação
+Wire Notes Line
+	700  4450 700  650
+Wire Notes Line
+	700  650  4800 650
+Wire Notes Line
+	4800 650  4800 4450
+Wire Notes Line
+	4800 4450 700  4450
+Text Notes 750  650  0    50   ~ 0
+PIC18F4550-I/PT
 $EndSCHEMATC

Commit message: .
Connections:
- no-connect marks 0 -> 2
Changed lines of the file:
@@
 Text Notes 750  650  0    50   ~ 0
 PIC18F4550-I/PT
+NoConn ~ 1100 5850
+NoConn ~ 400  4700
 $EndSCHEMATC

Commit message: .
Parts:
- added D? (x4): LED, symbol Device:LED
Connections:
- net USB_D-: now reaches U?.18 (D-)
- net USB_D-: now also J?.2 (D-)
- net USB_D+: now reaches U?.19 (D+)
- net USB_D+: now also J?.3 (D+)
Changed lines of the file:
@@
 NoConn ~ 1100 5850
 NoConn ~ 400  4700
+Text Label 1700 5450 0    50   ~ 0
+USB_D+
+Text Label 1700 5550 0    50   ~ 0
+USB_D-
+Wire Wire Line
+	1500 5450 1700 5450
+Wire Wire Line
+	1500 5550 1700 5550
+Text Label 9200 1300 0    50   ~ 0
+USB_D+
+Text Label 9200 1500 0    50   ~ 0
+USB_D-
+Wire Wire Line
+	9050 1300 9200 1300
+Wire Wire Line
+	9050 1500 9200 1500
+$Comp
+L Device:LED D?
+U 1 1 60A81084
+P 8500 5150
+F 0 "D?" H 8493 4895 50  0000 C CNN
+F 1 "LED" H 8493 4986 50  0000 C CNN
+F 2 "" H 8500 5150 50  0001 C CNN
+F 3 "~" H 8500 5150 50  0001 C CNN
+	1    8500 5150
+	-1   0    0    1
+$EndComp
+$Comp
+L Device:LED D?
+U 1 1 60A84FEF
+P 8500 5500
+F 0 "D?" H 8493 5245 50  0000 C CNN
+F 1 "LED" H 8493 5336 50  0000 C CNN
+F 2 "" H 8500 5500 50  0001 C CNN
+F 3 "~" H 8500 5500 50  0001 C CNN
+	1    8500 5500
+	-1   0    0    1
+$EndComp
+$Comp
+L Device:LED D?
+U 1 1 60A859F9
+P 8500 5850
+F 0 "D?" H 8493 5595 50  0000 C CNN
+F 1 "LED" H 8493 5686 50  0000 C CNN
+F 2 "" H 8500 5850 50  0001 C CNN
+F 3 "~" H 8500 5850 50  0001 C CNN
+	1    8500 5850
+	-1   0    0    1
+$EndComp
+$Comp
+L Device:LED D?
+U 1 1 60A86409
+P 8500 6200
+F 0 "D?" H 8493 5945 50  0000 C CNN
+F 1 "LED" H 8493 6036 50  0000 C CNN
+F 2 "" H 8500 6200 50  0001 C CNN
+F 3 "~" H 8500 6200 50  0001 C CNN
+	1    8500 6200
+	-1   0    0    1
+$EndComp
+Wire Notes Line
+	8000 4500 9500 4500
+Wire Notes Line
+	9500 4500 9500 6400
+Wire Notes Line
+	9500 6400 8000 6400
+Wire Notes Line
+	8000 6400 8000 4500
 $EndSCHEMATC

Commit message: .
Parts:
- added D_PWR: LED, symbol Device:LED
- added J?: Jack-DC, symbol Connector:Jack-DC
- added R_LED_1, R_LED_2: 100, symbol Device:R_US
- added R_LED_PWR: 15, symbol Device:R_US
- gave numbers to parts that had none: 2
Connections:
- net GNDREF: now also D?.1 (K), D?.1 (K), Escrita_USB.1 (K), Leitura_USB.1 (K), D_PWR.1 (K), J?.2
- net VCC: now also J?.1
- net Vcc_5v: now also R_LED_PWR.2; no longer U?.1 (VDD)
- net PIC_Rx: now reaches U?.1 (SDO/RX/DT/RC7)
- net PIC_Rx: now also U?.10 (TX)
- net Interrupt_timer: now reaches U?.10 (RB2/AN8/INT2/VMO)
- net RTS_Conversor: now reaches U?.11 (RB3/AN9/CCP2/VPO)
- net RTS_Conversor: now also U?.11 (RTS)
- net VUSB_3.3v: now reaches U?.37 (VUSB)
- net VUSB_3.3v: now also U?.1 (VDD)
- net PIC_Tx: now reaches U?.44 (TX/CK/RC6)
- net PIC_Tx: now also U?.12 (RX)
- net USB_T_Led: now reaches U?.5 (GP7/TxLED)
- net USB_T_Led: now also R_LED_2.2
- net USB_R_Led: now reaches U?.6 (GP6/RxLED)
- net USB_R_Led: now also R_LED_1.2
- net at Leitura_USB.2 (A): now also R_LED_1.1
- net at Escrita_USB.2 (A): now also R_LED_2.1
- new net: D_PWR.2 (A), R_LED_PWR.1
Other:
- moved on the sheet: D?, Escrita_USB, Leitura_USB

Commit message: .
Parts:
- R_LED_PWR: value 15 -> 200
Changed lines of the file:
@@
 P 8700 5950
 F 0 "R_LED_PWR" V 8495 5950 50  0001 C CNN
-F 1 "15" V 8587 5950 50  0000 C CNN
+F 1 "200" V 8587 5950 50  0000 C CNN
 F 2 "" V 8740 5940 50  0001 C CNN
 F 3 "~" H 8700 5950 50  0001 C CNN

Commit message: teste
Parts:
- added C?: CTRIM, symbol Device:CTRIM
- added J?: Conn_01x10_Female, symbol Connector:Conn_01x10_Female
- added J?: Conn_01x10_Male, symbol Connector:Conn_01x10_Male
- added J?: Screw_Terminal_01x02, symbol Connector:Screw_Terminal_01x02
- added RV?: R_POT_TRIM, symbol Device:R_POT_TRIM
- added SW?: SW_Push, symbol Switch:SW_Push
- added U?: RC1602A, Display:RC1602A, symbol Display_Character:RC1602A
Changed lines of the file:
@@
 Wire Notes Line
 	700  6700 700  7600
+$Comp
+L Device:R_POT_TRIM RV?
+U 1 1 60AACFA5
+P 15500 2250
+F 0 "RV?" H 15430 2296 50  0000 R CNN
+F 1 "R_POT_TRIM" H 15430 2205 50  0000 R CNN
+F 2 "" H 15500 2250 50  0001 C CNN
+F 3 "~" H 15500 2250 50  0001 C CNN
+	1    15500 2250
+	1    0    0    -1
+$EndComp
+$Comp
+L Device:CTRIM C?
+U 1 1 60AAF1CA
+P 15800 2250
+F 0 "C?" H 15916 2296 50  0000 L CNN
+F 1 "CTRIM" H 15916 2205 50  0000 L CNN
+F 2 "" H 15800 2250 50  0001 C CNN
+F 3 "~" H 15800 2250 50  0001 C CNN
+	1    15800 2250
+	1    0    0    -1
+$EndComp
+$Comp
+L Connector:Conn_01x10_Female J?
+U 1 1 60AB1231
+P 15150 1450
+F 0 "J?" H 15178 1426 50  0000 L CNN
+F 1 "Conn_01x10_Female" H 15178 1335 50  0000 L CNN
+F 2 "" H 15150 1450 50  0001 C CNN
+F 3 "~" H 15150 1450 50  0001 C CNN
+	1    15150 1450
+	1    0    0    -1
+$EndComp
+$Comp
+L Connector:Conn_01x10_Male J?
+U 1 1 60AB2595
+P 14600 1450
+F 0 "J?" H 14708 2031 50  0000 C CNN
+F 1 "Conn_01x10_Male" H 14708 1940 50  0000 C CNN
+F 2 "" H 14600 1450 50  0001 C CNN
+F 3 "~" H 14600 1450 50  0001 C CNN
+	1    14600 1450
+	1    0    0    -1
+$EndComp
+$Comp
+L Switch:SW_Push SW?
+U 1 1 60AB901B
+P 14700 2350
+F 0 "SW?" H 14700 2635 50  0000 C CNN
+F 1 "SW_Push" H 14700 2544 50  0000 C CNN
+F 2 "" H 14700 2550 50  0001 C CNN
+F 3 "~" H 14700 2550 50  0001 C CNN
+	1    14700 2350
+	1    0    0    -1
+$EndComp
+$Comp
+L Connector:Screw_Terminal_01x02 J?
+U 1 1 60ABE90B
+P 15150 600
+F 0 "J?" H 15230 592 50  0000 L CNN
+F 1 "Screw_Terminal_01x02" H 15230 501 50  0000 L CNN
+F 2 "" H 15150 600 50  0001 C CNN
+F 3 "~" H 15150 600 50  0001 C CNN
+	1    15150 600
+	1    0    0    -1
+$EndComp
+$Comp
+L Display_Character:RC1602A U?
+U 1 1 60AE4362
+P 17450 1200
+F 0 "U?" H 17450 2081 50  0000 C CNN
+F 1 "RC1602A" H 17450 1990 50  0000 C CNN
+F 2 "Display:RC1602A" H 17550 400 50  0001 C CNN
+F 3 "http://www.raystar-optronics.com/down.php?ProID=18" H 17550 1100 50  0001 C CNN
+	1    17450 1200
+	1    0    0    -1
+$EndComp
 $EndSCHEMATC

Commit message: Revert "teste"
This reverts commit ae6c77bb40d1ae6f6efaeae59efb69416e5190d8.
Parts:
- removed C?: CTRIM, symbol Device:CTRIM
- removed J?: Conn_01x10_Female, symbol Connector:Conn_01x10_Female
- removed J?: Conn_01x10_Male, symbol Connector:Conn_01x10_Male
- removed J?: Screw_Terminal_01x02, symbol Connector:Screw_Terminal_01x02
- removed RV?: R_POT_TRIM, symbol Device:R_POT_TRIM
- removed SW?: SW_Push, symbol Switch:SW_Push
- removed U?: RC1602A, Display:RC1602A, symbol Display_Character:RC1602A
Changed lines of the file:
@@
 Wire Notes Line
 	700  6700 700  7600
-$Comp
-L Device:R_POT_TRIM RV?
-U 1 1 60AACFA5
-P 15500 2250
-F 0 "RV?" H 15430 2296 50  0000 R CNN
-F 1 "R_POT_TRIM" H 15430 2205 50  0000 R CNN
-F 2 "" H 15500 2250 50  0001 C CNN
-F 3 "~" H 15500 2250 50  0001 C CNN
-	1    15500 2250
-	1    0    0    -1
-$EndComp
-$Comp
-L Device:CTRIM C?
-U 1 1 60AAF1CA
-P 15800 2250
-F 0 "C?" H 15916 2296 50  0000 L CNN
-F 1 "CTRIM" H 15916 2205 50  0000 L CNN
-F 2 "" H 15800 2250 50  0001 C CNN
-F 3 "~" H 15800 2250 50  0001 C CNN
-	1    15800 2250
-	1    0    0    -1
-$EndComp
-$Comp
-L Connector:Conn_01x10_Female J?
-U 1 1 60AB1231
-P 15150 1450
-F 0 "J?" H 15178 1426 50  0000 L CNN
-F 1 "Conn_01x10_Female" H 15178 1335 50  0000 L CNN
-F 2 "" H 15150 1450 50  0001 C CNN
-F 3 "~" H 15150 1450 50  0001 C CNN
-	1    15150 1450
-	1    0    0    -1
-$EndComp
-$Comp
-L Connector:Conn_01x10_Male J?
-U 1 1 60AB2595
-P 14600 1450
-F 0 "J?" H 14708 2031 50  0000 C CNN
-F 1 "Conn_01x10_Male" H 14708 1940 50  0000 C CNN
-F 2 "" H 14600 1450 50  0001 C CNN
-F 3 "~" H 14600 1450 50  0001 C CNN
-	1    14600 1450
-	1    0    0    -1
-$EndComp
-$Comp
-L Switch:SW_Push SW?
-U 1 1 60AB901B
-P 14700 2350
-F 0 "SW?" H 14700 2635 50  0000 C CNN
-F 1 "SW_Push" H 14700 2544 50  0000 C CNN
-F 2 "" H 14700 2550 50  0001 C CNN
-F 3 "~" H 14700 2550 50  0001 C CNN
-	1    14700 2350
-	1    0    0    -1
-$EndComp
-$Comp
-L Connector:Screw_Terminal_01x02 J?
-U 1 1 60ABE90B
-P 15150 600
-F 0 "J?" H 15230 592 50  0000 L CNN
-F 1 "Screw_Terminal_01x02" H 15230 501 50  0000 L CNN
-F 2 "" H 15150 600 50  0001 C CNN
-F 3 "~" H 15150 600 50  0001 C CNN
-	1    15150 600
-	1    0    0    -1
-$EndComp
-$Comp
-L Display_Character:RC1602A U?
-U 1 1 60AE4362
-P 17450 1200
-F 0 "U?" H 17450 2081 50  0000 C CNN
-F 1 "RC1602A" H 17450 1990 50  0000 C CNN
-F 2 "Display:RC1602A" H 17550 400 50  0001 C CNN
-F 3 "http://www.raystar-optronics.com/down.php?ProID=18" H 17550 1100 50  0001 C CNN
-	1    17450 1200
-	1    0    0    -1
-$EndComp
 $EndSCHEMATC

Commit message: .
Parts:
- D_PWR_GREEN: renamed from D_PWR; value LED -> G_LED
Connections:
- net VUSB_3.3v: no longer U?.1 (VDD)
- net Vcc_5v: now also U?.1 (VDD)
- net CTS_Conversor: now reaches U?.38 (SPP0/RD0)
- net CTS_Conversor: now also U?.13 (CTS)
Changed lines of the file:
@@
 $Descr A4 11693 8268
 encoding utf-8
-Sheet 1 3
+Sheet 1 4
 Title ""
 Date ""
@@
 VUSB_3.3v
 Text GLabel 7900 950  0    50   Input ~ 0
-VUSB_3.3v
+Vcc_5v
 Wire Wire Line
 	7900 950  8050 950
@@
 $EndComp
 $Comp
-L Device:LED D_PWR
+L Device:LED D_PWR_GREEN
 U 1 1 60A99312
 P 9050 5950
-F 0 "D_PWR" H 9043 5787 50  0000 C CNN
-F 1 "LED" H 9043 5786 50  0001 C CNN
+F 0 "D_PWR_GREEN" H 9043 5787 50  0000 C CNN
+F 1 "G_LED" H 9043 5786 50  0001 C CNN
 F 2 "" H 9050 5950 50  0001 C CNN
 F 3 "~" H 9050 5950 50  0001 C CNN
@@
 Wire Notes Line
 	700  6700 700  7600
+Text Label 7100 1700 2    50   ~ 0
+CTS_Conversor
+Text Label 4150 2450 0    50   ~ 0
+CTS_Conversor
+Wire Wire Line
+	4100 2450 4150 2450
+$Comp
+L power:GNDREF #PWR?
+U 1 1 60AAEC4B
+P 8500 950
+F 0 "#PWR?" H 8500 700 50  0001 C CNN
+F 1 "GNDREF" H 8505 777 50  0000 C CNN
+F 2 "" H 8500 950 50  0001 C CNN
+F 3 "" H 8500 950 50  0001 C CNN
+	1    8500 950
+	1    0    0    -1
+$EndComp
+$Sheet
+S 9200 2250 500  300
+U 60AB2F80
+F0 "Ocilador_Conversor" 50
+F1 "Ocilador_Conversor.sch" 50
+$EndSheet
+Wire Wire Line
+	7100 1700 7250 1700
 $EndSCHEMATC
