File: KiCad/Projeto_PBLE01.sch (KiCad schematic (older format))
At the start: 13 parts

Commit message: .
Parts:
- added Cref: 1pF, symbol Device:C
- renumbered R_LED_PWR to G_LED_PWR
Connections:
- net labels added: RST_Conversor
- wire segments 60 -> 64
- no-connect marks 2 -> 7
Other:
- moved on the sheet: U?
Changed lines of the file:
@@
 $Descr A4 11693 8268
 encoding utf-8
-Sheet 1 4
+Sheet 1 5
 Title ""
 Date ""
@@
 L Interface_USB:MCP2200-I-SO U?
 U 1 1 609EF1C2
-P 8150 1900
-F 0 "U?" H 8150 1011 50  0000 C CNN
-F 1 "MCP2200-I-SO" H 8150 920 50  0000 C CNN
-F 2 "Package_SO:SOIC-20W_7.5x12.8mm_P1.27mm" H 8150 750 50  0001 C CNN
-F 3 "http://ww1.microchip.com/downloads/en/DeviceDoc/200022228D.pdf" H 8150 900 50  0001 C CNN
-	1    8150 1900
+P 9000 1750
+F 0 "U?" H 9000 861 50  0000 C CNN
+F 1 "MCP2200-I-SO" H 9000 770 50  0000 C CNN
+F 2 "Package_SO:SOIC-20W_7.5x12.8mm_P1.27mm" H 9000 600 50  0001 C CNN
+F 3 "http://ww1.microchip.com/downloads/en/DeviceDoc/200022228D.pdf" H 9000 750 50  0001 C CNN
+	1    9000 1750
 	1    0    0    -1
 $EndComp
@@
 L power:GNDREF #PWR?
 U 1 1 60A4860B
-P 8150 2950
-F 0 "#PWR?" H 8150 2700 50  0001 C CNN
-F 1 "GNDREF" H 8155 2777 50  0000 C CNN
-F 2 "" H 8150 2950 50  0001 C CNN
-F 3 "" H 8150 2950 50  0001 C CNN
-	1    8150 2950
-	1    0    0    -1
-$EndComp
-Wire Wire Line
-	8150 2700 8150 2950
+P 9000 2800
+F 0 "#PWR?" H 9000 2550 50  0001 C CNN
+F 1 "GNDREF" H 9005 2627 50  0000 C CNN
+F 2 "" H 9000 2800 50  0001 C CNN
+F 3 "" H 9000 2800 50  0001 C CNN
+	1    9000 2800
+	1    0    0    -1
+$EndComp
+Wire Wire Line
+	9000 2550 9000 2800
 Wire Wire Line
 	1200 6100 1200 5850
@@
 	1800 5250 1500 5250
 Wire Wire Line
-	8050 950  8050 1100
+	8900 800  8900 950
 $Sheet
 S 5500 1500 800  400
@@
 PIC18F4550-I/PT
 NoConn ~ 1100 5850
-NoConn ~ 400  4700
 Text Label 1700 5450 0    50   ~ 0
 USB_D+
@@
 Wire Wire Line
 	1500 5550 1700 5550
-Text Label 9200 1300 0    50   ~ 0
+Text Label 10050 1150 0    50   ~ 0
 USB_D+
-Text Label 9200 1500 0    50   ~ 0
+Text Label 10050 1350 0    50   ~ 0
 USB_D-
 Wire Wire Line
-	9050 1300 9200 1300
-Wire Wire Line
-	9050 1500 9200 1500
+	9900 1150 10050 1150
+Wire Wire Line
+	9900 1350 10050 1350
 $Comp
 L Device:LED Leitura_USB
@@
 Wire Wire Line
 	1550 2650 1700 2650
-Text Label 7150 2400 2    50   ~ 0
+Text Label 8000 2250 2    50   ~ 0
 USB_R_Led
-Text Label 7150 2500 2    50   ~ 0
+Text Label 8000 2350 2    50   ~ 0
 USB_T_Led
 Wire Wire Line
-	7150 2400 7250 2400
-Wire Wire Line
-	7150 2500 7250 2500
+	8000 2250 8100 2250
+Wire Wire Line
+	8000 2350 8100 2350
 Text Label 8500 4750 2    50   ~ 0
 USB_R_Led
@@
 Text GLabel 4200 2250 2    50   Input ~ 0
 VUSB_3.3v
-Text GLabel 7900 950  0    50   Input ~ 0
+Text GLabel 8750 800  0    50   Input ~ 0
 Vcc_5v
 Wire Wire Line
-	7900 950  8050 950
+	8750 800  8900 800
 Wire Wire Line
 	4200 2250 4100 2250
@@
 L power:GNDREF #PWR?
 U 1 1 60A9311E
-P 9300 6250
-F 0 "#PWR?" H 9300 6000 50  0001 C CNN
-F 1 "GNDREF" H 9305 6077 50  0000 C CNN
-F 2 "" H 9300 6250 50  0001 C CNN
-F 3 "" H 9300 6250 50  0001 C CNN
-	1    9300 6250
+P 9300 6100
+F 0 "#PWR?" H 9300 5850 50  0001 C CNN
+F 1 "GNDREF" H 9305 5927 50  0000 C CNN
+F 2 "" H 9300 6100 50  0001 C CNN
+F 3 "" H 9300 6100 50  0001 C CNN
+	1    9300 6100
 	1    0    0    -1
 $EndComp
@@
 U 1 1 60A9C520
 P 8700 4750
-F 0 "R_LED_1" V 8587 4750 50  0001 C CNN
-F 1 "100" V 8587 4750 50  0000 C CNN
+F 0 "R_LED_1" V 8587 4750 50  0000 C CNN
+F 1 "100" V 8587 4750 50  0001 C CNN
 F 2 "" V 8740 4740 50  0001 C CNN
 F 3 "~" H 8700 4750 50  0001 C CNN
@@
 U 1 1 60A9D43E
 P 8700 5050
-F 0 "R_LED_2" V 8495 5050 50  0001 C CNN
-F 1 "100" V 8587 5050 50  0000 C CNN
+F 0 "R_LED_2" V 8495 5050 50  0000 C CNN
+F 1 "100" V 8587 5050 50  0001 C CNN
 F 2 "" V 8740 5040 50  0001 C CNN
 F 3 "~" H 8700 5050 50  0001 C CNN
@@
 $EndComp
 $Comp
-L Device:R_US R_LED_PWR
+L Device:R_US G_LED_PWR
 U 1 1 60A9E08E
-P 8700 5950
-F 0 "R_LED_PWR" V 8495 5950 50  0001 C CNN
-F 1 "200" V 8587 5950 50  0000 C CNN
-F 2 "" V 8740 5940 50  0001 C CNN
-F 3 "~" H 8700 5950 50  0001 C CNN
-	1    8700 5950
+P 8550 5950
+F 0 "G_LED_PWR" V 8345 5950 50  0000 C CNN
+F 1 "200" V 8437 5950 50  0001 C CNN
+F 2 "" V 8590 5940 50  0001 C CNN
+F 3 "~" H 8550 5950 50  0001 C CNN
+	1    8550 5950
 	0    1    1    0
 $EndComp
-Text GLabel 8450 5950 0    50   Input ~ 0
+Text GLabel 8400 5950 0    50   Input ~ 0
 Vcc_5v
-Wire Wire Line
-	8450 5950 8550 5950
-Wire Wire Line
-	8850 5950 8900 5950
 Wire Wire Line
 	9200 4750 9300 4750
@@
 Wire Wire Line
 	9200 5950 9300 5950
-Connection ~ 9300 5950
-Wire Wire Line
-	9300 5950 9300 6250
 Wire Wire Line
 	8850 4750 8900 4750
@@
 Wire Wire Line
 	4100 1950 4250 1950
-Text Label 7100 1400 2    50   ~ 0
+Text Label 7950 1250 2    50   ~ 0
 PIC_Tx
-Text Label 7100 1500 2    50   ~ 0
+Text Label 7950 1350 2    50   ~ 0
 PIC_Rx
 Wire Wire Line
-	7100 1500 7250 1500
-Wire Wire Line
-	7250 1400 7100 1400
-Text Label 7100 1600 2    50   ~ 0
+	7950 1350 8100 1350
+Wire Wire Line
+	8100 1250 7950 1250
+Text Label 7950 1450 2    50   ~ 0
 RTS_Conversor
 Wire Wire Line
-	7100 1600 7250 1600
+	7950 1450 8100 1450
 Text Label 1550 2750 2    50   ~ 0
 RTS_Conversor
@@
 Wire Notes Line
 	700  6700 700  7600
-Text Label 7100 1700 2    50   ~ 0
+Text Label 7950 1550 2    50   ~ 0
 CTS_Conversor
 Text Label 4150 2450 0    50   ~ 0
@@
 L power:GNDREF #PWR?
 U 1 1 60AAEC4B
-P 8500 950
-F 0 "#PWR?" H 8500 700 50  0001 C CNN
-F 1 "GNDREF" H 8505 777 50  0000 C CNN
-F 2 "" H 8500 950 50  0001 C CNN
-F 3 "" H 8500 950 50  0001 C CNN
-	1    8500 950
+P 9400 800
+F 0 "#PWR?" H 9400 550 50  0001 C CNN
+F 1 "GNDREF" H 9405 627 50  0000 C CNN
+F 2 "" H 9400 800 50  0001 C CNN
+F 3 "" H 9400 800 50  0001 C CNN
+	1    9400 800
 	1    0    0    -1
 $EndComp
 $Sheet
-S 9200 2250 500  300
+S 10050 2100 500  300
 U 60AB2F80
 F0 "Ocilador_Conversor" 50
 F1 "Ocilador_Conversor.sch" 50
+F2 "X1" B L 10050 2150 50
+F3 "X2" B L 10050 2350 50
 $EndSheet
 Wire Wire Line
-	7100 1700 7250 1700
+	7950 1550 8100 1550
+Wire Wire Line
+	10050 2150 9900 2150
+Wire Wire Line
+	9900 2350 10050 2350
+Text Label 7950 1150 2    50   ~ 0
+RST_Conversor
+Wire Wire Line
+	7950 1150 8100 1150
+Text Label 4150 2550 0    50   ~ 0
+RST_Conversor
+Wire Wire Line
+	4100 2550 4150 2550
+NoConn ~ 8100 1650
+NoConn ~ 8100 1750
+NoConn ~ 8100 1850
+NoConn ~ 8100 1950
+NoConn ~ 8100 2050
+NoConn ~ 8100 2150
+$Comp
+L Device:C Cref
+U 1 1 60ACBD01
+P 9250 800
+F 0 "Cref" V 9090 800 50  0000 C CNN
+F 1 "1pF" V 9089 800 50  0001 C CNN
+F 2 "" H 9288 650 50  0001 C CNN
+F 3 "~" H 9250 800 50  0001 C CNN
+	1    9250 800
+	0    1    1    0
+$EndComp
+Wire Wire Line
+	9100 800  9100 950
+Wire Wire Line
+	9300 6100 9300 5950
+Connection ~ 9300 5950
+Wire Wire Line
+	8700 5950 8900 5950
+$Sheet
+S 5300 3000 750  1400
+U 60AF7D01
+F0 "LCD" 50
+F1 "LCD.sch" 50
+$EndSheet
 $EndSCHEMATC

Commit message: .
Parts:
- removed Cref: 1pF, symbol Device:C
- removed U?: MCP2200-I-SO, Package_SO:SOIC-20W_7.5x12.8mm_P1.27mm, symbol Interface_USB:MCP2200-I-SO
- added Analog_00, Analog_01: Screw_Terminal_01x02, symbol Connector:Screw_Terminal_01x02
- added C_Reset: 10u, symbol Device:C
- added R_Reset: 10k, symbol Device:R_US
- added Reset_Button: SW_Push, symbol Switch:SW_Push
- gave numbers to parts that had none: 1
Connections:
- net labels added: Analog_0, Analog_1, Analog_2, Analog_3, LCD_B0, LCD_B1, LCD_B2, LCD_B3, LCD_B4, LCD_B5, LCD_B6, LCD_B7, LCD_ENABLE, LCD_RS, LCD_RW, MCLR
- net labels removed: ICSP_MCLR, RST_Conversor
- wire segments 64 -> 94
- no-connect marks 7 -> 1
Other:
- note added: "Leds"
- note added: "Reset\n"
- moved on the sheet: D?, D_PWR_GREEN, Escrita_USB, G_LED_PWR, Leitura_USB, R_LED_1, R_LED_2

Commit message: .
Parts:
- added IO_Pins: Conn_01x08_Female, symbol Connector:Conn_01x08_Female
- added Source_Pins: Conn_01x02_Female, symbol Connector:Conn_01x02_Female
Connections:
- net labels added: IO_00, IO_01, IO_02, IO_03, IO_04, IO_05, IO_06
- wire segments 94 -> 110
Changed lines of the file:
@@
 Text Label 2900 5700 0    50   ~ 0
 ICSP_Data
-Text Label 1350 3050 2    50   ~ 0
+Text Label 1350 3350 2    50   ~ 0
 ICSP_Clk
-Text Label 1350 3150 2    50   ~ 0
+Text Label 1350 3450 2    50   ~ 0
 ICSP_Data
 Wire Wire Line
-	1350 3050 1700 3050
-Wire Wire Line
-	1350 3150 1700 3150
+	1350 3350 1700 3350
+Wire Wire Line
+	1350 3450 1700 3450
 Text Label 4200 3650 0    50   ~ 0
 MCLR
@@
 Wire Wire Line
 	4100 1750 4150 1750
+Text Label 4250 1550 0    50   ~ 0
+IO_01
+Text Label 4250 1450 0    50   ~ 0
+IO_00
+Text Label 4250 1650 0    50   ~ 0
+IO_02
+Text Label 4200 3350 0    50   ~ 0
+IO_03
+Text Label 4200 3450 0    50   ~ 0
+IO_04
+Text Label 4200 3550 0    50   ~ 0
+IO_05
+Wire Wire Line
+	4250 1450 4100 1450
+Wire Wire Line
+	4250 1550 4100 1550
+Wire Wire Line
+	4250 1650 4100 1650
+Wire Wire Line
+	4200 3350 4100 3350
+Wire Wire Line
+	4200 3450 4100 3450
+Wire Wire Line
+	4200 3550 4100 3550
+Text Label 4500 5700 0    50   ~ 0
+IO_01
+Text Label 4500 5800 0    50   ~ 0
+IO_00
+Text Label 4500 5600 0    50   ~ 0
+IO_02
+Wire Wire Line
+	4500 5800 4350 5800
+Wire Wire Line
+	4500 5700 4350 5700
+Wire Wire Line
+	4500 5600 4350 5600
+Text Label 4500 5500 0    50   ~ 0
+IO_03
+Text Label 4500 5400 0    50   ~ 0
+IO_04
+Text Label 4500 5300 0    50   ~ 0
+IO_05
+Wire Wire Line
+	4350 5500 4500 5500
+Wire Wire Line
+	4350 5400 4500 5400
+Wire Wire Line
+	4350 5300 4500 5300
+Text Label 1550 2850 2    50   ~ 0
+IO_06
+Wire Wire Line
+	1550 2850 1700 2850
+Text Label 4500 5200 0    50   ~ 0
+IO_06
+Wire Wire Line
+	4350 5200 4500 5200
+$Comp
+L Connector:Conn_01x08_Female IO_Pins
+U 1 1 60D32B7F
+P 4150 5500
+F 0 "IO_Pins" H 4042 4967 50  0000 C CNN
+F 1 "Conn_01x08_Female" H 4042 4966 50  0001 C CNN
+F 2 "" H 4150 5500 50  0001 C CNN
+F 3 "~" H 4150 5500 50  0001 C CNN
+	1    4150 5500
+	-1   0    0    1
+$EndComp
+$Comp
+L Connector:Conn_01x02_Female Source_Pins
+U 1 1 60D35570
+P 4150 6200
+F 0 "Source_Pins" H 4042 5967 50  0000 C CNN
+F 1 "Conn_01x02_Female" H 4042 5966 50  0001 C CNN
+F 2 "" H 4150 6200 50  0001 C CNN
+F 3 "~" H 4150 6200 50  0001 C CNN
+	1    4150 6200
+	-1   0    0    1
+$EndComp
+Text GLabel 4500 6100 2    50   BiDi ~ 0
+Vcc_5v
+Wire Wire Line
+	4350 6100 4500 6100
+$Comp
+L power:GNDREF #PWR?
+U 1 1 60D3D5A5
+P 4500 6200
+F 0 "#PWR?" H 4500 5950 50  0001 C CNN
+F 1 "GNDREF" H 4505 6027 50  0000 C CNN
+F 2 "" H 4500 6200 50  0001 C CNN
+F 3 "" H 4500 6200 50  0001 C CNN
+	1    4500 6200
+	1    0    0    -1
+$EndComp
+Wire Wire Line
+	4350 6200 4500 6200
 $EndSCHEMATC

Commit message: 24/05
Parts:
- removed ICSP_Pin: Conn_01x05_Male, symbol Connector:Conn_01x05_Male
- added B0, B1, B2, B3, B4: SW_Push, symbol Switch:SW_Push
- added ICSP_IO: Conn_01x06_Male, symbol Connector:Conn_01x06_Male
- added R_B0: 2k, symbol Device:R_US
- added R_B1: 330, symbol Device:R_US
- added R_B2: 620, symbol Device:R_US
- added R_B3: 1k, symbol Device:R_US
- added R_B4: 3.3k, symbol Device:R_US
- gave numbers to parts that had none: 2
Connections:
- net labels added: Analog_KB, ICSP_Enable, ICSP_RST
- wire segments 110 -> 124
- no-connect marks 1 -> 3
Other:
- note added: "Teclado"
- moved on the sheet: PWR_Source

Commit message: 25/05
Connections:
- net Analog_0: no longer Analog_00.1 (Pin_1)
- net Analog_1: no longer Analog_00.2 (Pin_2)
- net Analog_2: no longer Analog_01.1 (Pin_1)
- net Analog_3: no longer Analog_01.2 (Pin_2)
Other:
- moved on the sheet: Analog_00, Analog_01, ICSP_IO
Changed lines of the file:
@@
 $Descr A4 11693 8268
 encoding utf-8
-Sheet 1 6
+Sheet 1 8
 Title ""
 Date ""
@@
 Wire Wire Line
 	1800 5250 1500 5250
-Text Label 2850 5550 0    50   ~ 0
+Text Label 2750 5450 0    50   ~ 0
 ICSP_Clk
-Text Label 2850 5450 0    50   ~ 0
+Text Label 2750 5350 0    50   ~ 0
 ICSP_Data
 Text Label 1350 3350 2    50   ~ 0
@@
 L power:GNDREF #PWR0104
 U 1 1 60A5C611
-P 3450 5350
-F 0 "#PWR0104" H 3450 5100 50  0001 C CNN
-F 1 "GNDREF" H 3455 5177 50  0000 C CNN
-F 2 "" H 3450 5350 50  0001 C CNN
-F 3 "" H 3450 5350 50  0001 C CNN
-	1    3450 5350
-	1    0    0    -1
-$EndComp
-Text GLabel 3450 5250 2    50   Input ~ 0
+P 3350 5250
+F 0 "#PWR0104" H 3350 5000 50  0001 C CNN
+F 1 "GNDREF" H 3355 5077 50  0000 C CNN
+F 2 "" H 3350 5250 50  0001 C CNN
+F 3 "" H 3350 5250 50  0001 C CNN
+	1    3350 5250
+	1    0    0    -1
+$EndComp
+Text GLabel 3350 5150 2    50   Input ~ 0
 Vcc_5v
 Text Label 1550 2450 2    50   ~ 0
@@
 L Connector:Screw_Terminal_01x02 Analog_00
 U 1 1 60B32822
-P 3300 6200
-F 0 "Analog_00" H 3380 6146 50  0000 L CNN
-F 1 "Screw_Terminal_01x02" H 3380 6101 50  0001 L CNN
-F 2 "" H 3300 6200 50  0001 C CNN
-F 3 "~" H 3300 6200 50  0001 C CNN
-	1    3300 6200
+P 3250 5800
+F 0 "Analog_00" H 3330 5746 50  0000 L CNN
+F 1 "Screw_Terminal_01x02" H 3330 5701 50  0001 L CNN
+F 2 "" H 3250 5800 50  0001 C CNN
+F 3 "~" H 3250 5800 50  0001 C CNN
+	1    3250 5800
 	1    0    0    -1
 $EndComp
@@
 L Connector:Screw_Terminal_01x02 Analog_01
 U 1 1 60B35301
-P 2100 6200
-F 0 "Analog_01" H 2180 6146 50  0000 L CNN
-F 1 "Screw_Terminal_01x02" H 2018 5966 50  0001 C CNN
-F 2 "" H 2100 6200 50  0001 C CNN
-F 3 "~" H 2100 6200 50  0001 C CNN
-	1    2100 6200
+P 3250 6200
+F 0 "Analog_01" H 3330 6146 50  0000 L CNN
+F 1 "Screw_Terminal_01x02" H 3168 5966 50  0001 C CNN
+F 2 "" H 3250 6200 50  0001 C CNN
+F 3 "~" H 3250 6200 50  0001 C CNN
+	1    3250 6200
 	1    0    0    -1
 $EndComp
@@
 Text Label 1550 1750 2    50   ~ 0
 Analog_3
-Text Label 3000 6200 2    50   ~ 0
+Text Label 2450 5800 2    50   ~ 0
 Analog_0
-Text Label 3000 6300 2    50   ~ 0
+Text Label 2450 5900 2    50   ~ 0
 Analog_1
-Text Label 1800 6200 2    50   ~ 0
-Analog_2
-Text Label 1800 6300 2    50   ~ 0
-Analog_3
-Wire Wire Line
-	3100 6300 3000 6300
-Wire Wire Line
-	3100 6200 3000 6200
-Wire Wire Line
-	1900 6300 1800 6300
-Wire Wire Line
-	1900 6200 1800 6200
+Wire Wire Line
+	2550 5900 2450 5900
+Wire Wire Line
+	2550 5800 2450 5800
 $Comp
 L power:GNDREF #PWR0107
@@
 Wire Wire Line
 	1350 3650 1700 3650
-Text Label 2850 5150 0    50   ~ 0
+Text Label 2750 5050 0    50   ~ 0
 ICSP_RST
 $Comp
 L Connector:Conn_01x06_Male ICSP_IO
 U 1 1 60B42D02
-P 2400 5350
-F 0 "ICSP_IO" H 2508 5639 50  0000 C CNN
-F 1 "Conn_01x06_Male" H 2508 5640 50  0001 C CNN
-F 2 "" H 2400 5350 50  0001 C CNN
-F 3 "~" H 2400 5350 50  0001 C CNN
-	1    2400 5350
-	1    0    0    -1
-$EndComp
-Wire Wire Line
-	2600 5150 2850 5150
-Wire Wire Line
-	2600 5250 3450 5250
-Wire Wire Line
-	3450 5350 2600 5350
-Wire Wire Line
-	2600 5450 2850 5450
-Wire Wire Line
-	2600 5550 2850 5550
+P 2300 5250
+F 0 "ICSP_IO" H 2408 5539 50  0000 C CNN
+F 1 "Conn_01x06_Male" H 2408 5540 50  0001 C CNN
+F 2 "" H 2300 5250 50  0001 C CNN
+F 3 "~" H 2300 5250 50  0001 C CNN
+	1    2300 5250
+	1    0    0    -1
+$EndComp
+Wire Wire Line
+	2500 5050 2750 5050
+Wire Wire Line
+	2500 5150 3350 5150
+Wire Wire Line
+	3350 5250 2500 5250
+Wire Wire Line
+	2500 5350 2750 5350
+Wire Wire Line
+	2500 5450 2750 5450
 Text Label 1550 2950 2    50   ~ 0
 ICSP_Enable
 Wire Wire Line
 	1550 2950 1700 2950
-Text Label 2850 5650 0    50   ~ 0
+Text Label 2750 5550 0    50   ~ 0
 ICSP_Enable
 Wire Wire Line
-	2600 5650 2850 5650
+	2500 5550 2750 5550
 $Comp
 L Switch:SW_Push B0
@@
 Wire Wire Line
 	1550 1850 1700 1850
+$Sheet
+S 2550 5700 500  700
+U 60B29ED3
+F0 "LM358" 50
+F1 "LM358.sch" 50
+$EndSheet
+$Sheet
+S 6800 2550 700  550
+U 60B32A3D
+F0 "Potenciometro" 50
+F1 "Potenciometro.sch" 50
+F2 "Saida_Analog" B L 6800 2800 50
+$EndSheet
+Text Label 6700 2800 2    50   ~ 0
+Analog_2
+Wire Wire Line
+	6700 2800 6800 2800
 $EndSCHEMATC
