File: KiCad/Projeto_PBLE01.sch (KiCad schematic (older format))
At the start: 29 parts

Commit message: 26/05
Parts:
- added D1, D2: LED, symbol Device:LED
- added R_LED_1, R_LED_2, R_LED_3, R_LED_4: 100, symbol Device:R_US
- C_Reset: value 10u -> 10uF
- gave numbers to parts that had none: 2
- renumbered R_LED_1 to R_LED_USB_R, R_LED_2 to R_LED_USB_R
Connections:
- net Analog_3 is gone; now on net IO_02: MCU.22 (RA3/AN3/Vref+)
- net GNDREF: now also D1.1 (K), D2.1 (K)
- net IO_02: no longer MCU.36 (P1A/CCP1/RC2)
- net IO_04: now also MCU.16 (RB6/KBI2/PGC); no longer MCU.26 (CK2SPP/AN6/RE1)
- net IO_05: now also MCU.17 (RB7/KBI3/PGD); no longer MCU.27 (OESPP/AN7/RE2)
- net IO_06: now also MCU.26 (CK2SPP/AN6/RE1)
- net at D3.2 (A): now also R_LED_3.1
- net at D4.2 (A): now also R_LED_4.1
- net IO_07: now reaches IO_Pins.8 (Pin_8)
- net IO_07: now also MCU.27 (OESPP/AN7/RE2)
- new net: D1.2 (A), R_LED_1.1
- new net: D2.2 (A), R_LED_2.1
Other:
- note added: "PWR_FLAGs"
- note added: "Periféricos"
- moved on the sheet: Escrita_USB, Leitura_USB, R_LED_USB_R
Changed lines of the file:
@@
 Wire Notes Line
 	700  6500 700  4850
-Wire Notes Line
-	700  4850 5950 4850
 Text Notes 750  4850 0    50   ~ 0
 Saídas/entradas
-Wire Notes Line
-	2750 7550 700  7550
-Wire Notes Line
-	700  6650 2750 6650
 Text Notes 750  6650 0    50   ~ 0
 Alimentação
@@
 Wire Notes Line
 	4800 650  4800 4450
-Wire Notes Line
-	4800 4450 700  4450
 Text Notes 750  650  0    50   ~ 0
 PIC18F4550-I/PT
@@
 L Device:LED Leitura_USB
 U 1 1 60A81084
-P 10450 4700
-F 0 "Leitura_USB" H 10443 4537 50  0000 C CNN
-F 1 "LED" H 10443 4536 50  0001 C CNN
-F 2 "" H 10450 4700 50  0001 C CNN
-F 3 "~" H 10450 4700 50  0001 C CNN
-	1    10450 4700
+P 10450 4100
+F 0 "Leitura_USB" H 10443 3937 50  0000 C CNN
+F 1 "LED" H 10443 3936 50  0001 C CNN
+F 2 "" H 10450 4100 50  0001 C CNN
+F 3 "~" H 10450 4100 50  0001 C CNN
+	1    10450 4100
 	-1   0    0    1
 $EndComp
@@
 L Device:LED Escrita_USB
 U 1 1 60A84FEF
-P 10450 5000
-F 0 "Escrita_USB" H 10443 4837 50  0000 C CNN
-F 1 "LED" H 10443 4836 50  0001 C CNN
-F 2 "" H 10450 5000 50  0001 C CNN
-F 3 "~" H 10450 5000 50  0001 C CNN
-	1    10450 5000
+P 10450 4400
+F 0 "Escrita_USB" H 10443 4237 50  0000 C CNN
+F 1 "LED" H 10443 4236 50  0001 C CNN
+F 2 "" H 10450 4400 50  0001 C CNN
+F 3 "~" H 10450 4400 50  0001 C CNN
+	1    10450 4400
 	-1   0    0    1
 $EndComp
 $Comp
-L Device:LED D?
+L Device:LED D3
 U 1 1 60A859F9
 P 10450 5300
-F 0 "D?" H 10443 5137 50  0000 C CNN
+F 0 "D3" H 10443 5137 50  0000 C CNN
 F 1 "LED" H 10443 5136 50  0001 C CNN
 F 2 "" H 10450 5300 50  0001 C CNN
@@
 $EndComp
 $Comp
-L Device:LED D?
+L Device:LED D4
 U 1 1 60A86409
 P 10450 5600
-F 0 "D?" H 10443 5437 50  0000 C CNN
+F 0 "D4" H 10443 5437 50  0000 C CNN
 F 1 "LED" H 10443 5436 50  0001 C CNN
 F 2 "" H 10450 5600 50  0001 C CNN
@@
 $EndComp
 Wire Notes Line
-	9400 4450 10900 4450
-Wire Notes Line
-	10900 4450 10900 6350
-Wire Notes Line
 	10900 6350 9400 6350
-Wire Notes Line
-	9400 6350 9400 4450
 Text Label 1550 2650 2    50   ~ 0
 Interrupt_timer
 Wire Wire Line
 	1550 2650 1700 2650
-Text Label 9900 4700 2    50   ~ 0
+Text Label 9900 4100 2    50   ~ 0
 USB_R_Led
-Text Label 9900 5000 2    50   ~ 0
+Text Label 9900 4400 2    50   ~ 0
 USB_T_Led
 Text GLabel 4200 2250 2    50   Input ~ 0
@@
 $EndComp
 $Comp
-L Device:R_US R_LED_1
+L Device:R_US R_LED_USB_R
 U 1 1 60A9C520
-P 10100 4700
-F 0 "R_LED_1" V 9987 4700 50  0000 C CNN
-F 1 "100" V 9987 4700 50  0001 C CNN
-F 2 "" V 10140 4690 50  0001 C CNN
-F 3 "~" H 10100 4700 50  0001 C CNN
-	1    10100 4700
+P 10100 4100
+F 0 "R_LED_USB_R" V 9987 4100 50  0000 C CNN
+F 1 "100" V 9987 4100 50  0001 C CNN
+F 2 "" V 10140 4090 50  0001 C CNN
+F 3 "~" H 10100 4100 50  0001 C CNN
+	1    10100 4100
 	0    1    1    0
 $EndComp
@@
 Vcc_5v
 Wire Wire Line
-	10600 4700 10700 4700
-Wire Wire Line
-	10700 4700 10700 5000
-Wire Wire Line
-	10600 5000 10700 5000
-Connection ~ 10700 5000
-Wire Wire Line
-	10700 5000 10700 5300
-Wire Wire Line
-	10600 5300 10700 5300
-Connection ~ 10700 5300
-Wire Wire Line
-	10700 5300 10700 5600
+	10600 4100 10700 4100
+Wire Wire Line
+	10700 4100 10700 4400
+Wire Wire Line
+	10600 4400 10700 4400
+Connection ~ 10700 4400
+Wire Wire Line
+	10700 4400 10700 4700
 Wire Wire Line
 	10600 5600 10700 5600
@@
 	10600 5900 10700 5900
 Wire Wire Line
-	10250 4700 10300 4700
-Wire Wire Line
-	10250 5000 10300 5000
-Wire Wire Line
-	9900 4700 9950 4700
-Wire Wire Line
-	9900 5000 9950 5000
+	10250 4100 10300 4100
+Wire Wire Line
+	10250 4400 10300 4400
+Wire Wire Line
+	9900 4100 9950 4100
+Wire Wire Line
+	9900 4400 9950 4400
 Text Label 4250 1950 0    50   ~ 0
 PIC_Tx
@@
 	1    0    0    -1
 $EndComp
-Wire Notes Line
-	2750 6650 2750 7550
-Wire Notes Line
-	700  6650 700  7550
 Text Label 8700 1350 2    50   ~ 0
 CTS_Conversor
@@
 Text Label 1550 1650 2    50   ~ 0
 Analog_2
-Text Label 1550 1750 2    50   ~ 0
-Analog_3
 Text Label 2450 5800 2    50   ~ 0
 Analog_0
@@
 P 7750 5650
 F 0 "C_Reset" H 7865 5696 50  0000 L CNN
-F 1 "10u" H 7865 5605 50  0000 L CNN
+F 1 "10uF" H 7865 5605 50  0000 L CNN
 F 2 "" H 7788 5500 50  0001 C CNN
 F 3 "~" H 7750 5650 50  0001 C CNN
@@
 Text Notes 7200 4550 0    50   ~ 0
 Reset\n
-Text Notes 9450 4450 0    50   ~ 0
+Text Notes 9450 3850 0    50   ~ 0
 Leds
 Text Label 10450 1000 0    50   ~ 0
@@
 F9 "D+" B R 10300 1000 50
 $EndSheet
-Wire Wire Line
-	1550 1750 1700 1750
 Wire Wire Line
 	1550 1650 1700 1650
@@
 Text Label 1550 1850 2    50   ~ 0
 IO_03
-Text Label 4200 3450 0    50   ~ 0
+Text Label 1550 3050 2    50   ~ 0
 IO_04
-Text Label 4200 3550 0    50   ~ 0
+Text Label 1550 3150 2    50   ~ 0
 IO_05
-Wire Wire Line
-	4200 3450 4100 3450
-Wire Wire Line
-	4200 3550 4100 3550
 Text Label 4500 5700 0    50   ~ 0
 IO_01
@@
 LCD_ENABLE
 Wire Wire Line
-	4250 1650 4100 1650
+	1550 1750 1700 1750
 Wire Wire Line
 	4250 1550 4100 1550
 Wire Wire Line
 	4250 1450 4100 1450
-Text Label 4250 1650 0    50   ~ 0
+Text Label 1550 1750 2    50   ~ 0
 IO_02
 Text Label 4250 1450 0    50   ~ 0
@@
 	1350 7100 1450 7100
 $Comp
-L Device:R_US R_LED_2
+L Device:R_US R_LED_USB_R
 U 1 1 60B24271
-P 10100 5000
-F 0 "R_LED_2" V 9987 5000 50  0000 C CNN
-F 1 "100" V 9987 5000 50  0001 C CNN
-F 2 "" V 10140 4990 50  0001 C CNN
-F 3 "~" H 10100 5000 50  0001 C CNN
-	1    10100 5000
+P 10100 4400
+F 0 "R_LED_USB_R" V 9987 4400 50  0000 C CNN
+F 1 "100" V 9987 4400 50  0001 C CNN
+F 2 "" V 10140 4390 50  0001 C CNN
+F 3 "~" H 10100 4400 50  0001 C CNN
+	1    10100 4400
 	0    1    1    0
 $EndComp
@@
 Wire Wire Line
 	6700 2800 6800 2800
+Wire Notes Line
+	3100 6650 3100 7650
+Wire Notes Line
+	3100 7650 700  7650
+Wire Notes Line
+	700  6650 3100 6650
+Wire Notes Line
+	700  6650 700  7650
+Wire Notes Line
+	6050 7650 6850 7650
+Wire Notes Line
+	6850 7650 6850 6650
+Wire Notes Line
+	6850 6650 6050 6650
+Wire Notes Line
+	6050 6650 6050 7650
+$Comp
+L power:PWR_FLAG #FLG0101
+U 1 1 60B3344B
+P 6250 6850
+F 0 "#FLG0101" H 6250 6925 50  0001 C CNN
+F 1 "PWR_FLAG" V 6250 6978 50  0000 L CNN
+F 2 "" H 6250 6850 50  0001 C CNN
+F 3 "~" H 6250 6850 50  0001 C CNN
+	1    6250 6850
+	0    1    1    0
+$EndComp
+$Comp
+L power:PWR_FLAG #FLG0102
+U 1 1 60B33451
+P 6250 7450
+F 0 "#FLG0102" H 6250 7525 50  0001 C CNN
+F 1 "PWR_FLAG" V 6250 7578 50  0000 L CNN
+F 2 "" H 6250 7450 50  0001 C CNN
+F 3 "~" H 6250 7450 50  0001 C CNN
+	1    6250 7450
+	0    1    1    0
+$EndComp
+$Comp
+L power:GNDREF #PWR0121
+U 1 1 60B33457
+P 6250 6850
+F 0 "#PWR0121" H 6250 6600 50  0001 C CNN
+F 1 "GNDREF" H 6255 6677 50  0000 C CNN
+F 2 "" H 6250 6850 50  0001 C CNN
+F 3 "" H 6250 6850 50  0001 C CNN
+	1    6250 6850
+	1    0    0    -1
+$EndComp
+$Comp
+L power:VCC #PWR0122
+U 1 1 60B3345D
+P 6250 7450
+F 0 "#PWR0122" H 6250 7300 50  0001 C CNN
+F 1 "VCC" H 6265 7623 50  0000 C CNN
+F 2 "" H 6250 7450 50  0001 C CNN
+F 3 "" H 6250 7450 50  0001 C CNN
+	1    6250 7450
+	1    0    0    -1
+$EndComp
+Wire Notes Line
+	9400 3850 10900 3850
+Wire Notes Line
+	10900 3850 10900 6350
+Wire Notes Line
+	9400 3850 9400 6350
+$Comp
+L Device:LED D1
+U 1 1 60B7D619
+P 10450 4700
+F 0 "D1" H 10443 4537 50  0000 C CNN
+F 1 "LED" H 10443 4536 50  0001 C CNN
+F 2 "" H 10450 4700 50  0001 C CNN
+F 3 "~" H 10450 4700 50  0001 C CNN
+	1    10450 4700
+	-1   0    0    1
+$EndComp
+$Comp
+L Device:LED D2
+U 1 1 60B7D61F
+P 10450 5000
+F 0 "D2" H 10443 4837 50  0000 C CNN
+F 1 "LED" H 10443 4836 50  0001 C CNN
+F 2 "" H 10450 5000 50  0001 C CNN
+F 3 "~" H 10450 5000 50  0001 C CNN
+	1    10450 5000
+	-1   0    0    1
+$EndComp
+Wire Wire Line
+	10600 4700 10700 4700
+Wire Wire Line
+	10600 5000 10700 5000
+$Comp
+L Device:R_US R_LED_1
+U 1 1 60B8546B
+P 10100 4700
+F 0 "R_LED_1" V 9987 4700 50  0000 C CNN
+F 1 "100" V 9987 4700 50  0001 C CNN
+F 2 "" V 10140 4690 50  0001 C CNN
+F 3 "~" H 10100 4700 50  0001 C CNN
+	1    10100 4700
+	0    1    1    0
+$EndComp
+$Comp
+L Device:R_US R_LED_2
+U 1 1 60B85471
+P 10100 5000
+F 0 "R_LED_2" V 9987 5000 50  0000 C CNN
+F 1 "100" V 9987 5000 50  0001 C CNN
+F 2 "" V 10140 4990 50  0001 C CNN
+F 3 "~" H 10100 5000 50  0001 C CNN
+	1    10100 5000
+	0    1    1    0
+$EndComp
+$Comp
+L Device:R_US R_LED_3
+U 1 1 60B8C6A6
+P 10100 5300
+F 0 "R_LED_3" V 9987 5300 50  0000 C CNN
+F 1 "100" V 9987 5300 50  0001 C CNN
+F 2 "" V 10140 5290 50  0001 C CNN
+F 3 "~" H 10100 5300 50  0001 C CNN
+	1    10100 5300
+	0    1    1    0
+$EndComp
+$Comp
+L Device:R_US R_LED_4
+U 1 1 60B8C6AC
+P 10100 5600
+F 0 "R_LED_4" V 9987 5600 50  0000 C CNN
+F 1 "100" V 9987 5600 50  0001 C CNN
+F 2 "" V 10140 5590 50  0001 C CNN
+F 3 "~" H 10100 5600 50  0001 C CNN
+	1    10100 5600
+	0    1    1    0
+$EndComp
+Wire Wire Line
+	10250 4700 10300 4700
+Wire Wire Line
+	10250 5000 10300 5000
+Wire Wire Line
+	10250 5300 10300 5300
+Wire Wire Line
+	10600 5300 10700 5300
+Connection ~ 10700 5300
+Wire Wire Line
+	10700 5300 10700 5600
+Wire Wire Line
+	10700 5000 10700 5300
+Connection ~ 10700 4700
+Wire Wire Line
+	10700 4700 10700 5000
+Connection ~ 10700 5000
+Wire Wire Line
+	10250 5600 10300 5600
+Wire Wire Line
+	1550 3050 1700 3050
+Text Label 4200 3450 0    50   ~ 0
+IO_06
+Wire Wire Line
+	4100 3450 4200 3450
+Wire Wire Line
+	1550 3150 1700 3150
+Text Label 4200 3550 0    50   ~ 0
+IO_07
+Wire Wire Line
+	4100 3550 4200 3550
+Text Label 4500 5100 0    50   ~ 0
+IO_07
+Wire Wire Line
+	4350 5100 4500 5100
+Wire Notes Line
+	4800 4450 700  4450
+Wire Notes Line
+	700  4850 5950 4850
+Wire Notes Line
+	10900 3500 5500 3500
+Wire Notes Line
+	5500 3500 5500 650
+Wire Notes Line
+	5500 650  10900 650
+Wire Notes Line
+	10900 650  10900 3500
+Text Notes 5550 650  0    50   ~ 0
+Periféricos
+Text Notes 6100 6650 0    50   ~ 0
+PWR_FLAGs
 $EndSCHEMATC

Commit message: PWM and minor changes
Filtro Butterworth e conexão dos LED's
Connections:
- net IO_00: no longer MCU.32 (T1OSO/T13CKI/RC0)
- net IO_01: no longer MCU.35 (~UOE~/CCP2/T1OSI/RC1)
- net IO_02: no longer MCU.22 (RA3/AN3/Vref+)
- net IO_03: no longer MCU.23 (RA4/T0CKI/C1OUT/RCV)
- net IO_06: no longer MCU.26 (CK2SPP/AN6/RE1)
- net IO_07: now also MCU.26 (CK2SPP/AN6/RE1); no longer MCU.27 (OESPP/AN7/RE2)
- net PWM_In: now reaches MCU.36 (P1A/CCP1/RC2)
- net IO_00_LED_1: now reaches R_LED_1.2
- net IO_00_LED_1: now also MCU.32 (T1OSO/T13CKI/RC0)
- net IO_01_LED_2: now reaches R_LED_2.2
- net IO_01_LED_2: now also MCU.35 (~UOE~/CCP2/T1OSI/RC1)
- net IO_02_LED_3: now reaches R_LED_3.2
- net IO_02_LED_3: now also MCU.22 (RA3/AN3/Vref+)
- net IO_03_LED_4: now reaches R_LED_4.2
- net IO_03_LED_4: now also MCU.23 (RA4/T0CKI/C1OUT/RCV)
- new net IO_08: MCU.27 (OESPP/AN7/RE2)
Other:
- note added: "PWM\n"
Changed lines of the file:
@@
 $Descr A4 11693 8268
 encoding utf-8
-Sheet 1 8
+Sheet 1 9
 Title ""
 Date ""
@@
 $EndSheet
 Text Label 1550 1850 2    50   ~ 0
-IO_03
+IO_03_LED_4
 Text Label 1550 3050 2    50   ~ 0
 IO_04
@@
 	4250 1450 4100 1450
 Text Label 1550 1750 2    50   ~ 0
-IO_02
+IO_02_LED_3
 Text Label 4250 1450 0    50   ~ 0
-IO_00
+IO_00_LED_1
 Text Label 4250 1550 0    50   ~ 0
-IO_01
+IO_01_LED_2
 Connection ~ 1350 7100
 Wire Wire Line
@@
 	1550 3050 1700 3050
 Text Label 4200 3450 0    50   ~ 0
-IO_06
+IO_07
 Wire Wire Line
 	4100 3450 4200 3450
@@
 	1550 3150 1700 3150
 Text Label 4200 3550 0    50   ~ 0
-IO_07
+IO_08
 Wire Wire Line
 	4100 3550 4200 3550
@@
 Text Notes 6100 6650 0    50   ~ 0
 PWR_FLAGs
+Wire Wire Line
+	4100 1650 4250 1650
+Text Label 4250 1650 0    50   ~ 0
+PWM
+Wire Notes Line
+	5150 3700 6900 3700
+Wire Notes Line
+	6900 3700 6900 4650
+Wire Notes Line
+	6900 4650 5150 4650
+Wire Notes Line
+	5150 4650 5150 3700
+Text Notes 5200 3700 0    50   ~ 0
+PWM\n
+$Sheet
+S 5600 3900 850  500
+U 60B33116
+F0 "filtro_PWM" 50
+F1 "filtro_PWM.sch" 50
+$EndSheet
+Text HLabel 5600 4150 2    50   Input ~ 0
+PWM_In
+Wire Wire Line
+	5600 4150 5350 4150
+Text HLabel 6450 4150 0    50   Output ~ 0
+PWM_Out
+Wire Wire Line
+	6450 4150 6700 4150
+Text Label 5350 4150 0    50   ~ 0
+PWM
+Text Label 6700 4150 0    50   ~ 0
+PWM_Out
+Wire Wire Line
+	9950 4700 9900 4700
+Text Label 9900 4700 2    50   ~ 0
+IO_00_LED_1
+Wire Wire Line
+	9950 5000 9900 5000
+Wire Wire Line
+	9950 5600 9900 5600
+Text Label 9900 5000 2    50   ~ 0
+IO_01_LED_2
+Wire Wire Line
+	9950 5300 9900 5300
+Text Label 9900 5300 2    50   ~ 0
+IO_02_LED_3
+Text Label 9900 5600 2    50   ~ 0
+IO_03_LED_4
 $EndSCHEMATC

Commit message: v1_final
Parts:
- removed IO_Pins: Conn_01x08_Female, symbol Connector:Conn_01x08_Female
- added IO_Pins1: Conn_01x09_Female, symbol Connector:Conn_01x09_Female
- added Led_Control1: SW_DIP_x04, symbol Switch:SW_DIP_x04
- renumbered Analog_00 to Analog_0, Analog_01 to Analog_1, C_Reset to C_Reset1, D_PWR_GREEN to D_PWR_GREEN1, Escrita_USB to Escrita_USB1, G_LED_PWR to G_LED_PWR1, ICSP_IO to ICSP_IO1, Leitura_USB to Leitura_USB1, MCU to MCU1, PWR_Source to PWR_Source1, Porta_USB to Porta_USB1, R_LED_USB_R to R_LED_USB_R1, R_LED_USB_R to R_LED_USB_R2, R_Reset to R_Reset1, Reset_Button to Reset_Button1, Source_Pins to Source_Pins1
Connections:
- net IO_00: now also MCU1.32 (T1OSO/T13CKI/RC0), IO_Pins1.1 (Pin_1), Led_Control1.1
- net IO_00_LED_1: now also Led_Control1.8; no longer MCU1.32 (T1OSO/T13CKI/RC0)
- net IO_01: now also MCU1.35 (~UOE~/CCP2/T1OSI/RC1), IO_Pins1.2 (Pin_2), Led_Control1.2
- net IO_01_LED_2: now also Led_Control1.7; no longer MCU1.35 (~UOE~/CCP2/T1OSI/RC1)
- net IO_02: now also MCU1.22 (RA3/AN3/Vref+), IO_Pins1.3 (Pin_3), Led_Control1.3
- net IO_02_LED_3: now also Led_Control1.6; no longer MCU1.22 (RA3/AN3/Vref+)
- net IO_03: now also MCU1.23 (RA4/T0CKI/C1OUT/RCV), IO_Pins1.4 (Pin_4), Led_Control1.4
- net IO_03_LED_4: now also Led_Control1.5; no longer MCU1.23 (RA4/T0CKI/C1OUT/RCV)
- net IO_04: now also MCU1.14 (RB4/AN11/KBI0/CSSPP), IO_Pins1.5 (Pin_5); no longer MCU1.16 (RB6/KBI2/PGC)
- net IO_05: now also MCU1.16 (RB6/KBI2/PGC), IO_Pins1.6 (Pin_6); no longer MCU1.17 (RB7/KBI3/PGD)
- net IO_06: now also MCU1.17 (RB7/KBI3/PGD), IO_Pins1.7 (Pin_7); no longer MCU1.14 (RB4/AN11/KBI0/CSSPP)
- net IO_07: now also IO_Pins1.8 (Pin_8)
- net IO_08: now also IO_Pins1.9 (Pin_9)
- net LM358/V-_1: now reaches Analog_0.1 (Pin_1)
- net LM358/V+_1: now reaches Analog_0.2 (Pin_2)
- net LM358/V-_2: now reaches Analog_1.1 (Pin_1)
- net LM358/V+_2: now reaches Analog_1.2 (Pin_2)
- net PWM_In renamed PWM
Other:
- note added: "Leds_Control"
- moved on the sheet: Analog_0, Analog_1, B0, B1, B2, B3, B4, C_Reset1, D1, D2, D3, D4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
