File: KiCad/Ocilador_Conversor.sch (KiCad schematic (older format))
At the start: 3 parts

Commit message: .
Changed lines of the file:
@@
 $Descr A4 11693 8268
 encoding utf-8
-Sheet 4 5
+Sheet 4 6
 Title ""
 Date ""
@@
 U 1 1 60AB6689
 P 5000 3500
-F 0 "Crystal_12MHz" V 4954 3631 50  0000 L CNN
+F 0 "Crystal_12MHz?" V 4954 3631 50  0000 L CNN
 F 1 "12MHz" V 5045 3631 50  0000 L CNN
 F 2 "" H 5000 3500 50  0001 C CNN
@@
 U 1 1 60AB901D
 P 5900 3400
-F 0 "C1" H 6015 3446 50  0000 L CNN
+F 0 "C?" H 6015 3446 50  0000 L CNN
 F 1 "22pF" H 6015 3355 50  0000 L CNN
 F 2 "" H 5938 3250 50  0001 C CNN
@@
 U 1 1 60AB99B5
 P 5500 3850
-F 0 "C2" V 5248 3850 50  0000 C CNN
+F 0 "C?" V 5248 3850 50  0000 C CNN
 F 1 "22pF" V 5339 3850 50  0000 C CNN
 F 2 "" H 5538 3700 50  0001 C CNN
