File: KiCad/Ocilador_Conversor.sch (KiCad schematic (older format))
At the start: 3 parts

Commit message: v1_final
Connections:
- net GNDREF: now also C2.2; no longer C2.1
- net X2: now also C2.1; no longer C2.2
Changed lines of the file:
@@
 P 5000 3500
 AR Path="/60AB2F80/60AB6689" Ref="Crystal_12MHz"  Part="1"
-AR Path="/60BE4F2F/60BE631A/60AB6689" Ref="Crystal_12MHz"  Part="1"
-F 0 "Crystal_12MHz" V 4954 3631 50  0000 L CNN
+AR Path="/60BE4F2F/60BE631A/60AB6689" Ref="Crystal_12MHz1"  Part="1"
+F 0 "Crystal_12MHz1" V 4954 3631 50  0000 L CNN
 F 1 "12MHz" V 5045 3631 50  0000 L CNN
 F 2 "" H 5000 3500 50  0001 C CNN
@@
 P 5900 3400
 AR Path="/60AB2F80/60AB901D" Ref="C1"  Part="1"
-AR Path="/60BE4F2F/60BE631A/60AB901D" Ref="C1"  Part="1"
-F 0 "C1" H 6015 3446 50  0000 L CNN
+AR Path="/60BE4F2F/60BE631A/60AB901D" Ref="C1_Cristal_12"  Part="1"
+F 0 "C1_Cristal_12" H 6015 3446 50  0000 L CNN
 F 1 "22pF" H 6015 3355 50  0000 L CNN
 F 2 "" H 5938 3250 50  0001 C CNN
@@
 P 5500 3850
 AR Path="/60AB2F80/60AB99B5" Ref="C2"  Part="1"
-AR Path="/60BE4F2F/60BE631A/60AB99B5" Ref="C2"  Part="1"
-F 0 "C2" V 5248 3850 50  0000 C CNN
+AR Path="/60BE4F2F/60BE631A/60AB99B5" Ref="C2__Cristal_12"  Part="1"
+F 0 "C2__Cristal_12" V 5248 3850 50  0000 C CNN
 F 1 "22pF" V 5339 3850 50  0000 C CNN
 F 2 "" H 5538 3700 50  0001 C CNN
 F 3 "~" H 5500 3850 50  0001 C CNN
 	1    5500 3850
-	0    1    1    0
+	0    -1   -1   0
 $EndComp
 Wire Wire Line

Commit message: adição de mais footprints
Parts:
- C1, C2: footprint (none) -> Capacitor_SMD:C_0805_2012Metric_Pad1.18x1.45mm_HandSolder
Changed lines of the file:
@@
 F 0 "C1_Cristal_12" H 6015 3446 50  0000 L CNN
 F 1 "22pF" H 6015 3355 50  0000 L CNN
-F 2 "" H 5938 3250 50  0001 C CNN
+F 2 "Capacitor_SMD:C_0805_2012Metric_Pad1.18x1.45mm_HandSolder" H 5938 3250 50  0001 C CNN
 F 3 "~" H 5900 3400 50  0001 C CNN
 	1    5900 3400
@@
 F 0 "C2__Cristal_12" V 5248 3850 50  0000 C CNN
 F 1 "22pF" V 5339 3850 50  0000 C CNN
-F 2 "" H 5538 3700 50  0001 C CNN
+F 2 "Capacitor_SMD:C_0805_2012Metric_Pad1.18x1.45mm_HandSolder" H 5538 3700 50  0001 C CNN
 F 3 "~" H 5500 3850 50  0001 C CNN
 	1    5500 3850

Commit message: pble_zip
Parts:
- Crystal_12MHz: footprint (none) -> Crystal:Crystal_HC49-4H_Vertical
Changed lines of the file:
@@
 F 0 "Crystal_12MHz1" V 4954 3631 50  0000 L CNN
 F 1 "12MHz" V 5045 3631 50  0000 L CNN
-F 2 "" H 5000 3500 50  0001 C CNN
+F 2 "Crystal:Crystal_HC49-4H_Vertical" H 5000 3500 50  0001 C CNN
 F 3 "~" H 5000 3500 50  0001 C CNN
 	1    5000 3500
