File: KiCad/Timer_I2C.sch (KiCad schematic (older format))
At the start: 5 parts

Commit message: .
Parts:
- added CX1, CX2: C, symbol Device:C
- added Cristal_AB38T_32.768KHZ: 32.768k, symbol Device:Crystal
- R_CLK, R_DATA: value R_US -> 10k
- gave numbers to parts that had none: 1
Connections:
- net GNDREF: now also CX1.2, CX2.1
- net X1_ocilador: no longer names the net of Timer_externo.1 (X1)
- net X1_ocilador: now also CX1.1, Cristal_AB38T_32.768KHZ.2
- net X2_ocilador: no longer names the net of Timer_externo.2 (X2)
- net X2_ocilador: now also CX2.2, Cristal_AB38T_32.768KHZ.1
Other:
- note removed: "Achar o valor de R_Clk"
- note removed: "achar o valor da capacitancia C_Vcc"
- note removed: "precisa saber a frequencia do cristal (ocilador) para sabermos a resistencia RD"
Changed lines of the file:
@@
 Wire Wire Line
 	4500 2500 4600 2500
-Text HLabel 4850 2900 2    50   BiDi ~ 0
-X1_ocilador
-Text HLabel 4850 3100 2    50   BiDi ~ 0
-X2_ocilador
-Wire Wire Line
-	4850 2900 4600 2900
-Wire Wire Line
-	4600 3100 4850 3100
 Text HLabel 3050 2800 0    50   Input ~ 0
 Serial_CLK
@@
 P 3400 2650
 F 0 "R_CLK" H 3468 2696 50  0000 L CNN
-F 1 "R_US" H 3468 2605 50  0000 L CNN
+F 1 "10k" H 3468 2605 50  0000 L CNN
 F 2 "" V 3440 2640 50  0001 C CNN
 F 3 "~" H 3400 2650 50  0001 C CNN
@@
 	3400 2400 3400 2500
 $Comp
-L Timer:MCP7940N-xSN U?
+L Timer:MCP7940N-xSN Timer_externo
 U 1 1 60A50A9A
 P 4200 3000
-F 0 "U?" H 4200 2511 50  0000 C CNN
+F 0 "Timer_externo" H 4200 2511 50  0000 C CNN
 F 1 "MCP7940N-xSN" H 4200 2420 50  0000 C CNN
 F 2 "" H 4200 3000 50  0001 C CNN
@@
 Wire Wire Line
 	3600 3100 3800 3100
-Text Notes 5050 2700 0    50   ~ 0
-precisa saber a frequencia do cristal (ocilador) para sabermos a resistencia RD
-Text Notes 4500 2100 0    50   ~ 0
-achar o valor da capacitancia C_Vcc
 Wire Wire Line
 	3750 2900 3800 2900
@@
 P 3750 2550
 F 0 "R_DATA" H 3818 2596 50  0000 L CNN
-F 1 "R_US" H 3818 2505 50  0000 L CNN
+F 1 "10k" H 3818 2505 50  0000 L CNN
 F 2 "" V 3790 2540 50  0001 C CNN
 F 3 "~" H 3750 2550 50  0001 C CNN
@@
 Wire Wire Line
 	3400 2400 3750 2400
-Text Notes 2950 2150 0    50   ~ 0
-Achar o valor de R_Clk
+Wire Wire Line
+	4600 2900 5550 2900
+Wire Wire Line
+	4600 3100 4600 3200
+Wire Wire Line
+	4600 3200 5550 3200
+$Comp
+L Device:Crystal Cristal_AB38T_32.768KHZ
+U 1 1 60A736EE
+P 5550 3050
+F 0 "Cristal_AB38T_32.768KHZ" V 5596 2919 50  0000 R CNN
+F 1 "32.768k" V 5505 2919 50  0000 R CNN
+F 2 "" H 5550 3050 50  0001 C CNN
+F 3 "~" H 5550 3050 50  0001 C CNN
+	1    5550 3050
+	0    -1   -1   0
+$EndComp
+$Comp
+L Device:C CX1
+U 1 1 60A761D7
+P 6800 3050
+F 0 "CX1" H 6915 3096 50  0000 L CNN
+F 1 "C" H 6915 3005 50  0000 L CNN
+F 2 "" H 6838 2900 50  0001 C CNN
+F 3 "~" H 6800 3050 50  0001 C CNN
+	1    6800 3050
+	1    0    0    -1
+$EndComp
+$Comp
+L Device:C CX2
+U 1 1 60A779E3
+P 5550 3350
+F 0 "CX2" H 5435 3304 50  0000 R CNN
+F 1 "C" H 5435 3395 50  0000 R CNN
+F 2 "" H 5588 3200 50  0001 C CNN
+F 3 "~" H 5550 3350 50  0001 C CNN
+	1    5550 3350
+	-1   0    0    1
+$EndComp
+Wire Wire Line
+	5550 2900 6800 2900
+Connection ~ 5550 2900
+Wire Wire Line
+	6800 3200 6800 3500
+Wire Wire Line
+	6800 3500 5550 3500
+$Comp
+L power:GNDREF #PWR?
+U 1 1 60A784D6
+P 5550 3500
+F 0 "#PWR?" H 5550 3250 50  0001 C CNN
+F 1 "GNDREF" H 5555 3327 50  0000 C CNN
+F 2 "" H 5550 3500 50  0001 C CNN
+F 3 "" H 5550 3500 50  0001 C CNN
+	1    5550 3500
+	1    0    0    -1
+$EndComp
+Connection ~ 5550 3500
 $EndSCHEMATC

Commit message: .
Parts:
- removed Cristal_AB38T_32.768KHZ: 32.768k, symbol Device:Crystal
- added Cristal-AB26T-32.768KHZ: 32.768kHz, Abracon-AB26T-32.768KHZ-*, symbol My_Lib:AB26T-32.768KHZ
Connections:
- net at CX1.1, Timer_externo.1 (X1): now also Cristal-AB26T-32.768KHZ.1
- net at CX2.2, Timer_externo.2 (X2): now also Cristal-AB26T-32.768KHZ.2
Changed lines of the file:
@@
 	3400 2400 3750 2400
-Wire Wire Line
-	4600 2900 5550 2900
 Wire Wire Line
 	4600 3100 4600 3200
 Wire Wire Line
 	4600 3200 5550 3200
-$Comp
-L Device:Crystal Cristal_AB38T_32.768KHZ
-U 1 1 60A736EE
-P 5550 3050
-F 0 "Cristal_AB38T_32.768KHZ" V 5596 2919 50  0000 R CNN
-F 1 "32.768k" V 5505 2919 50  0000 R CNN
-F 2 "" H 5550 3050 50  0001 C CNN
-F 3 "~" H 5550 3050 50  0001 C CNN
-	1    5550 3050
-	0    -1   -1   0
-$EndComp
 $Comp
 L Device:C CX1
@@
 $EndComp
 Wire Wire Line
-	5550 2900 6800 2900
-Connection ~ 5550 2900
-Wire Wire Line
 	6800 3200 6800 3500
 Wire Wire Line
@@
 $EndComp
 Connection ~ 5550 3500
+$Comp
+L My_Lib:AB26T-32.768KHZ Cristal-AB26T-32.768KHZ
+U 1 1 60A5D7A4
+P 5550 2900
+F 0 "Cristal-AB26T-32.768KHZ" V 5654 3028 50  0000 L CNN
+F 1 "32.768kHz" V 5745 3028 50  0000 L CNN
+F 2 "Abracon-AB26T-32.768KHZ-*" H 5550 3300 50  0001 L CNN
+F 3 "https://upverter.com/datasheet/e60e0d8762f6cc85b53388b76005bd605569ec5b.pdf" H 5550 3400 50  0001 L CNN
+F 4 "±20ppm" H 5550 3500 50  0001 L CNN "Frequency Tolerance"
+F 5 "Fundamental" H 5550 3600 50  0001 L CNN "Operating Mode"
+F 6 "Crys" H 5550 3700 50  0001 L CNN "category"
+F 7 "Crystals/Resonators/Oscillators" H 5550 3800 50  0001 L CNN "category 008acd80318bdb4d"
+F 8 "Uncategorized" H 5550 3900 50  0001 L CNN "category 6088ad82520dbb4f"
+F 9 "Passive Components" H 5550 4000 50  0001 L CNN "category 7542b8484461ae85"
+F 10 "Crystals" H 5550 4100 50  0001 L CNN "category 9afb57f1abf5413c"
+F 11 "32.768kHz ±20ppm Crystal 12.5pF 35 kOhm -10°C ~ 60°C Through Hole Cylindrical Can, Radial" H 5550 4200 50  0001 L CNN "digikey description"
+F 12 "535-9032-ND" H 5550 4300 50  0001 L CNN "digikey part number"
+F 13 "yes" H 5550 4400 50  0001 L CNN "lead free"
+F 14 "799e2e86d1baa452" H 5550 4500 50  0001 L CNN "library id"
+F 15 "Abracon" H 5550 4600 50  0001 L CNN "manufacturer"
+F 16 "through hole" H 5550 4700 50  0001 L CNN "mounting type"
+F 17 "815-AB26T-32.768KHZ" H 5550 4800 50  0001 L CNN "mouser part number"
+F 18 "2" H 5550 4900 50  0001 L CNN "num pins"
+F 19 "4ab983b7bf86957e" H 5550 5000 50  0001 L CNN "octopart part number"
+F 20 "RADIAL" H 5550 5100 50  0001 L CNN "package"
+F 21 "yes" H 5550 5200 50  0001 L CNN "rohs"
+F 22 "+60°C" H 5550 5300 50  0001 L CNN "temperature range high"
+F 23 "-10°C" H 5550 5400 50  0001 L CNN "temperature range low"
+F 24 "32.768kHz" H 5550 5500 50  0001 L CNN "frequency"
+F 25 "12.5pF" H 5550 5600 50  0001 L CNN "load capacitance"
+	1    5550 2900
+	0    1    1    0
+$EndComp
+Wire Wire Line
+	4600 2900 5550 2900
+Connection ~ 5550 2900
+Wire Wire Line
+	5550 2900 6800 2900
+Connection ~ 5550 3200
 $EndSCHEMATC

Commit message: .
Parts:
- CX1, CX2: value C -> 12.5pF
Changed lines of the file:
@@
 $Descr A4 11693 8268
 encoding utf-8
-Sheet 3 3
+Sheet 2 3
 Title ""
 Date ""
@@
 P 6800 3050
 F 0 "CX1" H 6915 3096 50  0000 L CNN
-F 1 "C" H 6915 3005 50  0000 L CNN
+F 1 "12.5pF" H 6915 3005 50  0000 L CNN
 F 2 "" H 6838 2900 50  0001 C CNN
 F 3 "~" H 6800 3050 50  0001 C CNN
@@
 P 5550 3350
 F 0 "CX2" H 5435 3304 50  0000 R CNN
-F 1 "C" H 5435 3395 50  0000 R CNN
+F 1 "12.5pF" H 5435 3395 50  0000 R CNN
 F 2 "" H 5588 3200 50  0001 C CNN
 F 3 "~" H 5550 3350 50  0001 C CNN

Commit message: .
Parts:
- removed C_Vcc: C, symbol Device:C
Changed lines of the file:
@@
 $Descr A4 11693 8268
 encoding utf-8
-Sheet 2 4
+Sheet 2 5
 Title ""
 Date ""
@@
 Text GLabel 4200 2350 1    50   Input ~ 0
 Vcc_5v
-Wire Wire Line
-	4200 2350 4200 2400
 $Comp
 L power:GNDREF #PWR?
@@
 Wire Wire Line
 	4300 2600 4300 2500
-Wire Wire Line
-	4300 2500 4500 2500
-$Comp
-L Device:C C_Vcc
-U 1 1 60A52D57
-P 4350 2400
-F 0 "C_Vcc" V 4098 2400 50  0000 C CNN
-F 1 "C" V 4189 2400 50  0000 C CNN
-F 2 "" H 4388 2250 50  0001 C CNN
-F 3 "~" H 4350 2400 50  0001 C CNN
-	1    4350 2400
-	0    1    1    0
-$EndComp
-Connection ~ 4200 2400
-Wire Wire Line
-	4200 2400 4200 2600
-Wire Wire Line
-	4500 2400 4500 2500
-Connection ~ 4500 2500
-Wire Wire Line
-	4500 2500 4600 2500
 Text HLabel 3050 2800 0    50   Input ~ 0
 Serial_CLK
@@
 	5550 2900 6800 2900
 Connection ~ 5550 3200
+Wire Wire Line
+	4200 2350 4200 2600
+Wire Wire Line
+	4300 2500 4600 2500
 $EndSCHEMATC

Commit message: Revert "Merge branch 'main' of https://github.com/EduardoDuenas/PBLE01 into main"
This reverts commit 9a71280a43de2c009adc09aa3a7293361a0fda06, reversing
changes made to ae6c77bb40d1ae6f6efaeae59efb69416e5190d8.
Parts:
- added C_Vcc: C, symbol Device:C
Connections:
- net GNDREF: now also C_Vcc.1
- net Vcc_5v: now also C_Vcc.2
Changed lines of the file:
@@
 $Descr A4 11693 8268
 encoding utf-8
-Sheet 2 5
+Sheet 2 3
 Title ""
 Date ""
@@
 Text GLabel 4200 2350 1    50   Input ~ 0
 Vcc_5v
+Wire Wire Line
+	4200 2350 4200 2400
 $Comp
 L power:GNDREF #PWR?
@@
 Wire Wire Line
 	4300 2600 4300 2500
+Wire Wire Line
+	4300 2500 4500 2500
+$Comp
+L Device:C C_Vcc
+U 1 1 60A52D57
+P 4350 2400
+F 0 "C_Vcc" V 4098 2400 50  0000 C CNN
+F 1 "C" V 4189 2400 50  0000 C CNN
+F 2 "" H 4388 2250 50  0001 C CNN
+F 3 "~" H 4350 2400 50  0001 C CNN
+	1    4350 2400
+	0    1    1    0
+$EndComp
+Connection ~ 4200 2400
+Wire Wire Line
+	4200 2400 4200 2600
+Wire Wire Line
+	4500 2400 4500 2500
+Connection ~ 4500 2500
+Wire Wire Line
+	4500 2500 4600 2500
 Text HLabel 3050 2800 0    50   Input ~ 0
 Serial_CLK
@@
 	5550 2900 6800 2900
 Connection ~ 5550 3200
-Wire Wire Line
-	4200 2350 4200 2600
-Wire Wire Line
-	4300 2500 4600 2500
 $EndSCHEMATC

Commit message: Safe_point
Parts:
- removed C_Vcc: C, symbol Device:C
Connections:
- wire segments 24 -> 23
Changed lines of the file:
@@
 $Descr A4 11693 8268
 encoding utf-8
-Sheet 2 3
+Sheet 2 5
 Title ""
 Date ""
@@
 Text GLabel 4200 2350 1    50   Input ~ 0
 Vcc_5v
-Wire Wire Line
-	4200 2350 4200 2400
 $Comp
 L power:GNDREF #PWR?
@@
 Wire Wire Line
 	4300 2500 4500 2500
-$Comp
-L Device:C C_Vcc
-U 1 1 60A52D57
-P 4350 2400
-F 0 "C_Vcc" V 4098 2400 50  0000 C CNN
-F 1 "C" V 4189 2400 50  0000 C CNN
-F 2 "" H 4388 2250 50  0001 C CNN
-F 3 "~" H 4350 2400 50  0001 C CNN
-	1    4350 2400
-	0    1    1    0
-$EndComp
-Connection ~ 4200 2400
-Wire Wire Line
-	4200 2400 4200 2600
 Wire Wire Line
 	4500 2400 4500 2500
@@
 	5550 2900 6800 2900
 Connection ~ 5550 3200
+Wire Wire Line
+	4200 2350 4200 2600
 $EndSCHEMATC

Commit message: .
Connections:
- wire segments 23 -> 21
Changed lines of the file:
@@
 $Descr A4 11693 8268
 encoding utf-8
-Sheet 2 5
+Sheet 2 6
 Title ""
 Date ""
@@
 Wire Wire Line
 	4300 2600 4300 2500
-Wire Wire Line
-	4300 2500 4500 2500
-Wire Wire Line
-	4500 2400 4500 2500
-Connection ~ 4500 2500
-Wire Wire Line
-	4500 2500 4600 2500
 Text HLabel 3050 2800 0    50   Input ~ 0
 Serial_CLK
@@
 Wire Wire Line
 	4200 2350 4200 2600
+Wire Wire Line
+	4300 2500 4600 2500
 $EndSCHEMATC
