File: KiCad/Timer_I2C.sch (KiCad schematic (older format))
At the start: 10 parts

Commit message: Valores dos capacitores CS
Parts:
- CS6: value 100n -> 100nF
Changed lines of the file:
@@
 P 4750 2300
 F 0 "CS6" V 4498 2300 50  0000 C CNN
-F 1 "100n" V 4589 2300 50  0000 C CNN
+F 1 "100nF" V 4589 2300 50  0000 C CNN
 F 2 "Capacitor_SMD:C_0805_2012Metric_Pad1.18x1.45mm_HandSolder" H 4788 2150 50  0001 C CNN
 F 3 "~" H 4750 2300 50  0001 C CNN
