File: KiCad/Retificador_de_tensão.sch (KiCad schematic (older format))
At the start: 4 parts

Commit message: v1_final
Parts:
- renumbered C1 to C1_Retificador1, C2 to C2_Retificador1, D1 to D_Schottky1, Retificador_de_tensão_5v to Retificador_de_tensão_5v1
Changed lines of the file:
@@
 	6250 3300 6100 3300
 $Comp
-L Device:C C1
+L Device:C C1_Retificador1
 U 1 1 60A126EF
 P 4100 3650
-F 0 "C1" H 4215 3696 50  0000 L CNN
+F 0 "C1_Retificador1" H 4215 3696 50  0000 L CNN
 F 1 "100n" H 4215 3605 50  0000 L CNN
 F 2 "" H 4138 3500 50  0001 C CNN
@@
 $EndComp
 $Comp
-L Device:C C2
+L Device:C C2_Retificador1
 U 1 1 60A1336B
 P 6100 3650
-F 0 "C2" H 6215 3696 50  0000 L CNN
+F 0 "C2_Retificador1" H 6215 3696 50  0000 L CNN
 F 1 "10u" H 6215 3605 50  0000 L CNN
 F 2 "" H 6138 3500 50  0001 C CNN
@@
 	4300 3050 4100 3050
 $Comp
-L Diode:1N5819 D1
+L Diode:1N5819 D_Schottky1
 U 1 1 60A5E713
 P 3750 3300
-F 0 "D1" H 3750 3083 50  0000 C CNN
+F 0 "D_Schottky1" H 3750 3083 50  0000 C CNN
 F 1 "1N5819" H 3750 3174 50  0000 C CNN
 F 2 "Diode_THT:D_DO-41_SOD81_P10.16mm_Horizontal" H 3750 3125 50  0001 C CNN
@@
 	3500 3300 3600 3300
 $Comp
-L My_Lib:LD1117DT50TR Retificador_de_tensão_5v
+L My_Lib:LD1117DT50TR Retificador_de_tensão_5v1
 U 1 1 60A5A48D
 P 4300 3200
-F 0 "Retificador_de_tensão_5v" H 5200 3587 60  0000 C CNN
+F 0 "Retificador_de_tensão_5v1" H 5200 3587 60  0000 C CNN
 F 1 "LD1117DT50TR" H 5200 3481 60  0000 C CNN
 F 2 "DPAK_STM" H 5200 3440 60  0001 C CNN
