File: KiCad/Retificador_de_tensão.sch (KiCad schematic (older format))
At the start: 4 parts

Commit message: adição departe dos footprints
Parts:
- Retificador_de_tensão_5v1: footprint DPAK_STM -> (none)
Changed lines of the file:
@@
 $Descr A4 11693 8268
 encoding utf-8
-Sheet 2 9
+Sheet 2 10
 Title ""
 Date ""
@@
 F 0 "Retificador_de_tensão_5v1" H 5200 3587 60  0000 C CNN
 F 1 "LD1117DT50TR" H 5200 3481 60  0000 C CNN
-F 2 "DPAK_STM" H 5200 3440 60  0001 C CNN
+F 2 "" H 5200 3440 60  0001 C CNN
 F 3 "" H 4300 3200 60  0000 C CNN
 	1    4300 3200

Commit message: adição de mais footprints
Parts:
- C1_Retificador1: footprint (none) -> Capacitor_SMD:C_0805_2012Metric_Pad1.18x1.45mm_HandSolder
Changed lines of the file:
@@
 F 0 "C1_Retificador1" H 4215 3696 50  0000 L CNN
 F 1 "100n" H 4215 3605 50  0000 L CNN
-F 2 "" H 4138 3500 50  0001 C CNN
+F 2 "Capacitor_SMD:C_0805_2012Metric_Pad1.18x1.45mm_HandSolder" H 4138 3500 50  0001 C CNN
 F 3 "~" H 4100 3650 50  0001 C CNN
 	1    4100 3650

Commit message: pble_zip
Parts:
- C2_Retificador1: footprint (none) -> Capacitor_Tantalum_SMD:CP_EIA-3216-18_Kemet-A_Pad1.58x1.35mm_HandSolder
- Retificador_de_tensão_5v1: footprint (none) -> Converter_ACDC:LD1117DT50TR
Changed lines of the file:
@@
 F 0 "C2_Retificador1" H 6215 3696 50  0000 L CNN
 F 1 "10u" H 6215 3605 50  0000 L CNN
-F 2 "" H 6138 3500 50  0001 C CNN
+F 2 "Capacitor_Tantalum_SMD:CP_EIA-3216-18_Kemet-A_Pad1.58x1.35mm_HandSolder" H 6138 3500 50  0001 C CNN
 F 3 "~" H 6100 3650 50  0001 C CNN
 	1    6100 3650
@@
 F 0 "Retificador_de_tensão_5v1" H 5200 3587 60  0000 C CNN
 F 1 "LD1117DT50TR" H 5200 3481 60  0000 C CNN
-F 2 "" H 5200 3440 60  0001 C CNN
+F 2 "Converter_ACDC:LD1117DT50TR" H 5200 3440 60  0001 C CNN
 F 3 "" H 4300 3200 60  0000 C CNN
 	1    4300 3200

Commit message: começo da pcb
Parts:
- Retificador_de_tensão_5v1: footprint Converter_ACDC:LD1117DT50TR -> My_Lib:LD1117DT50TR
Changed lines of the file:
@@
 F 0 "Retificador_de_tensão_5v1" H 5200 3587 60  0000 C CNN
 F 1 "LD1117DT50TR" H 5200 3481 60  0000 C CNN
-F 2 "Converter_ACDC:LD1117DT50TR" H 5200 3440 60  0001 C CNN
+F 2 "My_Lib:LD1117DT50TR" H 5200 3440 60  0001 C CNN
 F 3 "" H 4300 3200 60  0000 C CNN
 	1    4300 3200

Commit message: PCB resolução dos erros
Parts:
- Retificador_de_tensão_5v1: footprint My_Lib:LD1117DT50TR -> Package_TO_SOT_SMD:TO-252-3_TabPin2
Changed lines of the file:
@@
 F 0 "Retificador_de_tensão_5v1" H 5200 3587 60  0000 C CNN
 F 1 "LD1117DT50TR" H 5200 3481 60  0000 C CNN
-F 2 "My_Lib:LD1117DT50TR" H 5200 3440 60  0001 C CNN
+F 2 "Package_TO_SOT_SMD:TO-252-3_TabPin2" H 5200 3440 60  0001 C CNN
 F 3 "" H 4300 3200 60  0000 C CNN
 	1    4300 3200
