File: KiCad/Conversor_UART_USB.sch (KiCad schematic (older format))
At the start: 4 parts

Commit message: 26/05
Parts:
- renumbered C_Reset to C_Reset_Conversor
Changed lines of the file:
@@
 	2550 3000 2550 2900
 $Comp
-L Device:CP1 C_Reset
+L Device:CP1 C_Reset_Conversor
 U 1 1 60BE969F
 P 2550 2750
-F 0 "C_Reset" H 2665 2796 50  0000 L CNN
+F 0 "C_Reset_Conversor" H 2665 2796 50  0000 L CNN
 F 1 "1uF" H 2665 2705 50  0000 L CNN
 F 2 "" H 2550 2750 50  0001 C CNN

Commit message: v1_final
Parts:
- renumbered C_Reset_Conversor to C_Reset_Conversor1, Conversor_UART_USB to Conversor_UART_USB1
Changed lines of the file:
@@
 P 4950 3200
 AR Path="/60BE6306" Ref="U?"  Part="1"
-AR Path="/60BE4F2F/60BE6306" Ref="Conversor_UART_USB"  Part="1"
-F 0 "Conversor_UART_USB" H 4950 2311 50  0000 C CNN
+AR Path="/60BE4F2F/60BE6306" Ref="Conversor_UART_USB1"  Part="1"
+F 0 "Conversor_UART_USB1" H 4950 2311 50  0000 C CNN
 F 1 "MCP2200-I-SO" H 4950 2220 50  0000 C CNN
 F 2 "Package_SO:SOIC-20W_7.5x12.8mm_P1.27mm" H 4950 2050 50  0001 C CNN
@@
 	2550 3000 2550 2900
 $Comp
-L Device:CP1 C_Reset_Conversor
+L Device:CP1 C_Reset_Conversor1
 U 1 1 60BE969F
 P 2550 2750
-F 0 "C_Reset_Conversor" H 2665 2796 50  0000 L CNN
+F 0 "C_Reset_Conversor1" H 2665 2796 50  0000 L CNN
 F 1 "1uF" H 2665 2705 50  0000 L CNN
 F 2 "" H 2550 2750 50  0001 C CNN

Commit message: correção do RST do conversor
Parts:
- added R_RST1: 1k, symbol Device:R_US
Connections:
- net Vcc_5v: now also R_RST1.1
- net at C_Reset_Conversor1.1, Conversor_UART_USB1.4 (RST): now also R_RST1.2
Changed lines of the file:
@@
 Wire Wire Line
 	5850 2800 5950 2800
+Text GLabel 2550 2200 0    50   Input ~ 0
+Vcc_5v
+$Comp
+L Device:R_US R_RST1
+U 1 1 60C2C5EA
+P 2550 2350
+F 0 "R_RST1" H 2618 2396 50  0000 L CNN
+F 1 "1k" H 2618 2305 50  0000 L CNN
+F 2 "" V 2590 2340 50  0001 C CNN
+F 3 "~" H 2550 2350 50  0001 C CNN
+	1    2550 2350
+	1    0    0    -1
+$EndComp
+Wire Wire Line
+	2550 2500 2550 2600
+Connection ~ 2550 2600
 $EndSCHEMATC

Commit message: Finalização do esquemático
Connections:
- net Vcc_5v: no longer R_RST1.1
- new net Vbus: R_RST1.1
Changed lines of the file:
@@
 $Descr A4 11693 8268
 encoding utf-8
-Sheet 3 9
+Sheet 8 9
 Title ""
 Date ""
@@
 Wire Wire Line
 	5850 2800 5950 2800
-Text GLabel 2550 2200 0    50   Input ~ 0
-Vcc_5v
 $Comp
 L Device:R_US R_RST1
@@
 	2550 2500 2550 2600
 Connection ~ 2550 2600
+Text HLabel 2500 2200 0    50   UnSpc ~ 0
+Vbus
+Wire Wire Line
+	2500 2200 2550 2200
 $EndSCHEMATC

Commit message: adição departe dos footprints
Parts:
- R_RST1: footprint (none) -> Resistor_SMD:R_0805_2012Metric
Changed lines of the file:
@@
 $Descr A4 11693 8268
 encoding utf-8
-Sheet 8 9
+Sheet 8 10
 Title ""
 Date ""
@@
 F 0 "R_RST1" H 2618 2396 50  0000 L CNN
 F 1 "1k" H 2618 2305 50  0000 L CNN
-F 2 "" V 2590 2340 50  0001 C CNN
+F 2 "Resistor_SMD:R_0805_2012Metric" V 2590 2340 50  0001 C CNN
 F 3 "~" H 2550 2350 50  0001 C CNN
 	1    2550 2350
