File: KiCad/Cristal_20MHz.sch (KiCad schematic (older format))
At the start: 3 parts

Commit message: adição de mais footprints
Parts:
- CX1_20MHz1, CX2_20MHz1: footprint (none) -> Capacitor_SMD:C_0805_2012Metric_Pad1.18x1.45mm_HandSolder
Changed lines of the file:
@@
 F 0 "CX1_20MHz1" V 6598 2850 50  0000 C CNN
 F 1 "15pF" V 6689 2850 50  0000 C CNN
-F 2 "" H 6888 2700 50  0001 C CNN
+F 2 "Capacitor_SMD:C_0805_2012Metric_Pad1.18x1.45mm_HandSolder" H 6888 2700 50  0001 C CNN
 F 3 "~" H 6850 2850 50  0001 C CNN
 	1    6850 2850
@@
 F 0 "CX2_20MHz1" V 6598 3550 50  0000 C CNN
 F 1 "15pF" V 6689 3550 50  0000 C CNN
-F 2 "" H 6888 3400 50  0001 C CNN
+F 2 "Capacitor_SMD:C_0805_2012Metric_Pad1.18x1.45mm_HandSolder" H 6888 3400 50  0001 C CNN
 F 3 "~" H 6850 3550 50  0001 C CNN
 	1    6850 3550

Commit message: pble_zip
Parts:
- Cristal_20MHz1: footprint (none) -> Crystal:Crystal_HC49-4H_Vertical
Changed lines of the file:
@@
 F 0 "Cristal_20MHz1" V 6154 3331 50  0000 L CNN
 F 1 "20MHz" V 6245 3331 50  0000 L CNN
-F 2 "" H 6200 3200 50  0001 C CNN
+F 2 "Crystal:Crystal_HC49-4H_Vertical" H 6200 3200 50  0001 C CNN
 F 3 "~" H 6200 3200 50  0001 C CNN
 	1    6200 3200
