File: KiCad/LM358.sch (KiCad schematic (older format))
At the start: 1 part

Commit message: v1_final
Parts:
- added Ganho_AO_1, Ganho_AO_2: SW_DIP_x04, symbol Switch:SW_DIP_x04
- added R1_AO_1, R1_AO_2, R2_10k_AO_1, R2_10k_AO_2: 10k, symbol Device:R_US
- added R2_30k_2_AO_1, R2_30k_2_AO_2, R2_30k_3_AO_1, R2_30k_3_AO_2, R2_30k_AO_1, R2_30k_AO_2: 30k, symbol Device:R_US
- gave numbers to parts that had none: 1
Connections:
- net VUSB_3.3v: now also IC1.8 (VCC)
- net Out_1: now reaches IC1.1 (1OUT)
- net Out_1: now also Ganho_AO_1.1, R2_10k_AO_1.1
- net at IC1.2 (1IN-): now also Ganho_AO_1.5, Ganho_AO_1.6, Ganho_AO_1.7, Ganho_AO_1.8, R1_AO_1.1
- net V+_1: now reaches IC1.3 (1IN+)
- net V+_2: now reaches IC1.5 (2IN+)
- net at IC1.6 (2IN-): now also Ganho_AO_2.5, Ganho_AO_2.6, Ganho_AO_2.7, Ganho_AO_2.8, R1_AO_2.2
- net Out_2: now reaches IC1.7 (2OUT)
- net Out_2: now also Ganho_AO_2.1, R2_10k_AO_2.2
- new net: Ganho_AO_1.2, R2_10k_AO_1.2, R2_30k_AO_1.1
- new net: Ganho_AO_1.3, R2_30k_2_AO_1.1, R2_30k_AO_1.2
- new net: Ganho_AO_1.4, R2_30k_3_AO_1.2
- new net: R2_30k_2_AO_1.2, R2_30k_3_AO_1.1
- new net: Ganho_AO_2.2, R2_10k_AO_2.1, R2_30k_AO_2.1
- new net: Ganho_AO_2.3, R2_30k_2_AO_2.1, R2_30k_AO_2.2
- new net: Ganho_AO_2.4, R2_30k_3_AO_2.1
- new net: R2_30k_2_AO_2.2, R2_30k_3_AO_2.2
- new net V-_1: R1_AO_1.2
- new net V-_2: R1_AO_2.1

Commit message: correção da avaliação cruzada
Connections:
- net VUSB_3.3v renamed Vcc_5v
Other:
- note added: "Saturação 0,3v-3,3v"
Changed lines of the file:
@@
 	4650 3300 4850 3300
 Text GLabel 6100 3000 2    50   Input ~ 0
-VUSB_3.3v
+Vcc_5v
 $Comp
 L My_Lib:LM358 IC1
@@
 F 1 "LM358" H 5400 3174 50  0000 C CNN
 F 2 "SOP100P600X150-8N" H 5800 3100 50  0001 L CNN
-F 3 "https://datasheet.lcsc.com/szlcsc/1902201702_IDCHIP-LM358_C329455.pdf" H 5800 3000 50  0001 L CNN
+F 3 "https://www.onsemi.com/pdf/datasheet/lm358-d.pdf" H 5800 3000 50  0001 L CNN
 F 4 "Operational Amplifiers SOP-8 RoHS" H 5800 2900 50  0001 L CNN "Description"
 F 5 "1.5" H 5800 2800 50  0001 L CNN "Height"
@@
 Wire Wire Line
 	6600 3200 6950 3200
+Text Notes 5100 2600 0    50   ~ 0
+Saturação 0,3v-3,3v
 $EndSCHEMATC

Commit message: adição departe dos footprints
Parts:
- IC1: footprint SOP100P600X150-8N -> (none)
- R1_AO_1, R1_AO_2, R2_10k_AO_1, R2_10k_AO_2, R2_30k_2_AO_1, R2_30k_2_AO_2, R2_30k_3_AO_1, R2_30k_3_AO_2, R2_30k_AO_1, R2_30k_AO_2: footprint (none) -> Resistor_SMD:R_0805_2012Metric
Changed lines of the file:
@@
 $Descr A4 11693 8268
 encoding utf-8
-Sheet 7 9
+Sheet 7 10
 Title ""
 Date ""
@@
 F 0 "IC1" H 5400 3265 50  0000 C CNN
 F 1 "LM358" H 5400 3174 50  0000 C CNN
-F 2 "SOP100P600X150-8N" H 5800 3100 50  0001 L CNN
+F 2 "" H 5800 3100 50  0001 L CNN
 F 3 "https://www.onsemi.com/pdf/datasheet/lm358-d.pdf" H 5800 3000 50  0001 L CNN
 F 4 "Operational Amplifiers SOP-8 RoHS" H 5800 2900 50  0001 L CNN "Description"
@@
 F 0 "R1_AO_1" V 3945 3100 50  0001 C CNN
 F 1 "10k" V 4037 3100 50  0000 C CNN
-F 2 "" V 4190 3090 50  0001 C CNN
+F 2 "Resistor_SMD:R_0805_2012Metric" V 4190 3090 50  0001 C CNN
 F 3 "~" H 4150 3100 50  0001 C CNN
 	1    4150 3100
@@
 F 0 "R2_10k_AO_1" H 3418 1846 50  0001 L CNN
 F 1 "10k" H 3418 1800 50  0000 L CNN
-F 2 "" V 3390 1790 50  0001 C CNN
+F 2 "Resistor_SMD:R_0805_2012Metric" V 3390 1790 50  0001 C CNN
 F 3 "~" H 3350 1800 50  0001 C CNN
 	1    3350 1800
@@
 F 0 "R2_30k_AO_1" H 3418 2246 50  0001 L CNN
 F 1 "30k" H 3418 2200 50  0000 L CNN
-F 2 "" V 3390 2190 50  0001 C CNN
+F 2 "Resistor_SMD:R_0805_2012Metric" V 3390 2190 50  0001 C CNN
 F 3 "~" H 3350 2200 50  0001 C CNN
 	1    3350 2200
@@
 F 0 "R2_30k_2_AO_1" H 3418 2596 50  0001 L CNN
 F 1 "30k" H 3418 2550 50  0000 L CNN
-F 2 "" V 3390 2540 50  0001 C CNN
+F 2 "Resistor_SMD:R_0805_2012Metric" V 3390 2540 50  0001 C CNN
 F 3 "~" H 3350 2550 50  0001 C CNN
 	1    3350 2550
@@
 F 0 "R2_30k_3_AO_1" H 3668 2746 50  0001 L CNN
 F 1 "30k" V 3487 2700 50  0000 C CNN
-F 2 "" V 3640 2690 50  0001 C CNN
+F 2 "Resistor_SMD:R_0805_2012Metric" V 3640 2690 50  0001 C CNN
 F 3 "~" H 3600 2700 50  0001 C CNN
 	1    3600 2700
@@
 F 0 "R1_AO_2" V 6805 3600 50  0001 C CNN
 F 1 "10k" V 6487 3600 50  0000 C CNN
-F 2 "" V 6640 3590 50  0001 C CNN
+F 2 "Resistor_SMD:R_0805_2012Metric" V 6640 3590 50  0001 C CNN
 F 3 "~" H 6600 3600 50  0001 C CNN
 	1    6600 3600
@@
 F 0 "R2_10k_AO_2" H 8318 4496 50  0001 L CNN
 F 1 "10k" H 8182 4450 50  0000 R CNN
-F 2 "" V 8290 4440 50  0001 C CNN
+F 2 "Resistor_SMD:R_0805_2012Metric" V 8290 4440 50  0001 C CNN
 F 3 "~" H 8250 4450 50  0001 C CNN
 	1    8250 4450
@@
 F 0 "R2_30k_AO_2" H 8318 4096 50  0001 L CNN
 F 1 "30k" H 8318 4050 50  0000 L CNN
-F 2 "" V 8290 4040 50  0001 C CNN
+F 2 "Resistor_SMD:R_0805_2012Metric" V 8290 4040 50  0001 C CNN
 F 3 "~" H 8250 4050 50  0001 C CNN
 	1    8250 4050
@@
 F 0 "R2_30k_2_AO_2" H 8318 3746 50  0001 L CNN
 F 1 "30k" H 8318 3700 50  0000 L CNN
-F 2 "" V 8290 3690 50  0001 C CNN
+F 2 "Resistor_SMD:R_0805_2012Metric" V 8290 3690 50  0001 C CNN
 F 3 "~" H 8250 3700 50  0001 C CNN
 	1    8250 3700
@@
 F 0 "R2_30k_3_AO_2" H 8068 3596 50  0001 L CNN
 F 1 "30k" V 8113 3550 50  0000 C CNN
-F 2 "" V 8040 3540 50  0001 C CNN
+F 2 "Resistor_SMD:R_0805_2012Metric" V 8040 3540 50  0001 C CNN
 F 3 "~" H 8000 3550 50  0001 C CNN
 	1    8000 3550

Commit message: pble_zip
Parts:
- Ganho_AO_1, Ganho_AO_2: footprint (none) -> Button_Switch_THT:DIP4PIN
- IC1: footprint (none) -> Package_SO:SOIC-8_3.9x4.9mm_P1.27mm
Changed lines of the file:
@@
 F 0 "IC1" H 5400 3265 50  0000 C CNN
 F 1 "LM358" H 5400 3174 50  0000 C CNN
-F 2 "" H 5800 3100 50  0001 L CNN
+F 2 "Package_SO:SOIC-8_3.9x4.9mm_P1.27mm" H 5800 3100 50  0001 L CNN
 F 3 "https://www.onsemi.com/pdf/datasheet/lm358-d.pdf" H 5800 3000 50  0001 L CNN
 F 4 "Operational Amplifiers SOP-8 RoHS" H 5800 2900 50  0001 L CNN "Description"
@@
 F 0 "Ganho_AO_1" H 4150 2975 50  0000 C CNN
 F 1 "SW_DIP_x04" H 4150 2976 50  0001 C CNN
-F 2 "" H 4150 2600 50  0001 C CNN
+F 2 "Button_Switch_THT:DIP4PIN" H 4150 2600 50  0001 C CNN
 F 3 "~" H 4150 2600 50  0001 C CNN
 	1    4150 2600
@@
 F 0 "Ganho_AO_2" H 7450 3375 50  0000 C CNN
 F 1 "SW_DIP_x04" H 7450 4026 50  0001 C CNN
-F 2 "" H 7450 3650 50  0001 C CNN
+F 2 "Button_Switch_THT:DIP4PIN" H 7450 3650 50  0001 C CNN
 F 3 "~" H 7450 3650 50  0001 C CNN
 	1    7450 3650

Commit message: começo da pcb
Parts:
- Ganho_AO_1, Ganho_AO_2: footprint Button_Switch_THT:DIP4PIN -> My_Lib:DIP4PIN
Changed lines of the file:
@@
 F 0 "Ganho_AO_1" H 4150 2975 50  0000 C CNN
 F 1 "SW_DIP_x04" H 4150 2976 50  0001 C CNN
-F 2 "Button_Switch_THT:DIP4PIN" H 4150 2600 50  0001 C CNN
+F 2 "My_Lib:DIP4PIN" H 4150 2600 50  0001 C CNN
 F 3 "~" H 4150 2600 50  0001 C CNN
 	1    4150 2600
@@
 F 0 "Ganho_AO_2" H 7450 3375 50  0000 C CNN
 F 1 "SW_DIP_x04" H 7450 4026 50  0001 C CNN
-F 2 "Button_Switch_THT:DIP4PIN" H 7450 3650 50  0001 C CNN
+F 2 "My_Lib:DIP4PIN" H 7450 3650 50  0001 C CNN
 F 3 "~" H 7450 3650 50  0001 C CNN
 	1    7450 3650
