File: KiCad/Potenciometro.sch (KiCad schematic (older format))
At the start: 2 parts

Commit message: v1_final
Parts:
- renumbered POT to POT1, SW_POT to SW_POT1
Changed lines of the file:
@@
 $EndDescr
 $Comp
-L Device:R_POT_US POT
+L Device:R_POT_US POT1
 U 1 1 60B34708
 P 4000 3100
-F 0 "POT" H 3932 3146 50  0000 R CNN
+F 0 "POT1" H 3932 3146 50  0000 R CNN
 F 1 "10k" H 3932 3055 50  0000 R CNN
 F 2 "" H 4000 3100 50  0001 C CNN
@@
 $EndComp
 $Comp
-L Switch:SW_DIP_x01 SW_POT
+L Switch:SW_DIP_x01 SW_POT1
 U 1 1 60B35938
 P 4000 2650
-F 0 "SW_POT" V 3954 2780 50  0000 L CNN
+F 0 "SW_POT1" V 3954 2780 50  0000 L CNN
 F 1 "SW_DIP_x01" V 4045 2780 50  0000 L CNN
 F 2 "" H 4000 2650 50  0001 C CNN

Commit message: adição de mais footprints
Parts:
- POT1: footprint (none) -> LED_SMD:LED_2010_5025Metric
Changed lines of the file:
@@
 F 0 "POT1" H 3932 3146 50  0000 R CNN
 F 1 "10k" H 3932 3055 50  0000 R CNN
-F 2 "" H 4000 3100 50  0001 C CNN
+F 2 "LED_SMD:LED_2010_5025Metric" H 4000 3100 50  0001 C CNN
 F 3 "~" H 4000 3100 50  0001 C CNN
 	1    4000 3100

Commit message: pble_zip
Parts:
- SW_POT1: footprint (none) -> Button_Switch_THT:DIP1PIN
Changed lines of the file:
@@
 F 0 "SW_POT1" V 3954 2780 50  0000 L CNN
 F 1 "SW_DIP_x01" V 4045 2780 50  0000 L CNN
-F 2 "" H 4000 2650 50  0001 C CNN
+F 2 "Button_Switch_THT:DIP1PIN" H 4000 2650 50  0001 C CNN
 F 3 "~" H 4000 2650 50  0001 C CNN
 	1    4000 2650

Commit message: começo da pcb
Parts:
- POT1: footprint LED_SMD:LED_2010_5025Metric -> Potentiometer_THT:Potentiometer_Piher_T-16H_Single_Horizontal
- SW_POT1: footprint Button_Switch_THT:DIP1PIN -> My_Lib:DIP1PIN
Changed lines of the file:
@@
 F 0 "POT1" H 3932 3146 50  0000 R CNN
 F 1 "10k" H 3932 3055 50  0000 R CNN
-F 2 "LED_SMD:LED_2010_5025Metric" H 4000 3100 50  0001 C CNN
+F 2 "Potentiometer_THT:Potentiometer_Piher_T-16H_Single_Horizontal" H 4000 3100 50  0001 C CNN
 F 3 "~" H 4000 3100 50  0001 C CNN
 	1    4000 3100
@@
 F 0 "SW_POT1" V 3954 2780 50  0000 L CNN
 F 1 "SW_DIP_x01" V 4045 2780 50  0000 L CNN
-F 2 "Button_Switch_THT:DIP1PIN" H 4000 2650 50  0001 C CNN
+F 2 "My_Lib:DIP1PIN" H 4000 2650 50  0001 C CNN
 F 3 "~" H 4000 2650 50  0001 C CNN
 	1    4000 2650
